File: PCBs/Left_Main/Left_Main.kicad_sch (KiCad schematic)
At the start: 0 parts

Commit message: wip
Parts:
- added C3, C7: 100nF, symbol Device:C_Small
- added J1: Conn_IDC_Right_To_Left, symbol System_Connectors:Conn_IDC_Right_To_Left
- added J10: Rotary switch pins 1, symbol Connector:Screw_Terminal_01x07
- added J11: Future expansion, symbol Connector_Generic:Conn_02x13_Odd_Even
- added J2: Encoder inputs B, symbol Connector:Screw_Terminal_01x08
- added J6: Encoder inputs A, symbol Connector:Screw_Terminal_01x08
- added J7: Analog inputs, symbol Connector:Screw_Terminal_01x08
- added R1: 100, symbol Device:R_Small
- added U2: MCP23017_SP, Package_DIP:DIP-28_W7.62mm, symbol Interface_Expansion:MCP23017_SP
- added U5: 74HC4051, symbol 74xx:74HC4051
- added U7: ULN2003A, symbol Transistor_Array:ULN2003A
Connections:
- new net: J7.1 (Pin_1), U5.13 (A0)
- new net: J7.2 (Pin_2), U5.14 (A1)
- new net: J7.3 (Pin_3), U5.15 (A2)
- new net: J7.4 (Pin_4), U5.12 (A3)
- new net: J7.5 (Pin_5), U5.1 (A4)
- new net: J7.6 (Pin_6), U5.5 (A5)
- new net: J7.7 (Pin_7), U5.2 (A6)
- new net: J7.8 (Pin_8), U5.4 (A7)
- new net: J1., J1.24 (ANA_DA), U5.3 (A)
- new net: J1.10 (IOX_INT), J11.10 (Pin_10), U2.20 (INTA)
- new net: J1.12 (I2C_SCL), J11.12 (Pin_12), U2.12 (SCK)
- new net: J1.14 (I2C_SDA), J11.14 (Pin_14), U2.13 (SDA)
- new net: J1.16 (ANA_S0), J11.16 (Pin_16), U5.11 (S0)
- new net: J1.18 (ANA_S1), J11.18 (Pin_18), U5.10 (S1)
- new net: J1.20 (ANA_S2), J11.20 (Pin_20), U5.9 (S2)
- new net: J1.22 (RSW_MD), U7.1 (I1), U7.2 (I2), U7.3 (I3), U7.4 (I4), U7.5 (I5), U7.6 (I6), U7.7 (I7)
- new net: J1.4 (IN_DTM), R1.1
- new net: J6.1 (Pin_1), U2.21 (GPA0)
- new net: J6.2 (Pin_2), U2.22 (GPA1)
- new net: J6.3 (Pin_3), U2.23 (GPA2)
- new net: J6.4 (Pin_4), U2.24 (GPA3)
- new net: J6.5 (Pin_5), U2.25 (GPA4)
- new net: J6.6 (Pin_6), U2.26 (GPA5)
- new net: J6.7 (Pin_7), U2.27 (GPA6)
- new net: J6.8 (Pin_8), U2.28 (GPA7)
- new net: J2.1 (Pin_1), U2.1 (GPB0)
- new net: J2.2 (Pin_2), U2.2 (GPB1)
- new net: J2.3 (Pin_3), U2.3 (GPB2)
- new net: J2.4 (Pin_4), U2.4 (GPB3)
- new net: J2.5 (Pin_5), U2.5 (GPB4)
- new net: J2.6 (Pin_6), U2.6 (GPB5)
- new net: J2.7 (Pin_7), U2.7 (GPB6)
- new net: J2.8 (Pin_8), U2.8 (GPB7)
- new net: J10.1 (Pin_1), U7.16 (O1)
- new net: J10.2 (Pin_2), U7.15 (O2)
- new net: J10.3 (Pin_3), U7.14 (O3)
- new net: J10.4 (Pin_4), U7.13 (O4)
- new net: J10.5 (Pin_5), U7.12 (O5)
- new net: J10.6 (Pin_6), U7.11 (O6)
- new net: J10.7 (Pin_7), U7.10 (O7)
- new net +5V: C3.2, C7.1, J1.2 (5V), J11.2 (Pin_2), U2.16 (A1), U2.18 (~{RESET}), U2.9 (VDD), U5.16 (VCC)
- new net GND: C3.1, C7.2, J1.1 (GND_1), J1.11 (GND_6), J1.13 (GND_7), J1.15 (GND_8), J1.17 (GND_9), J1.19 (GND_10), J1.21 (GND_11), J1.23 (GND_12), J1.25 (GND_13), J1.3 (GND_2), J1.5 (GND_3), J1.7 (GND_4), J1.9 (GND_5), J11.1 (Pin_1), J11.11 (Pin_11), J11.13 (Pin_13), J11.15 (Pin_15), J11.17 (Pin_17), J11.19 (Pin_19), J11.21 (Pin_21), J11.23 (Pin_23), J11.25 (Pin_25), J11.3 (Pin_3), J11.5 (Pin_5), J11.7 (Pin_7), J11.9 (Pin_9), U2.10 (VSS), U2.15 (A0), U2.17 (A2), U5.6 (~{E}), U5.7 (VEE), U5.8 (GND), U7.8 (GND)
- new net Input shift register 1/CP: J1.6 (IN_CP), J11.6 (Pin_6)
- new net Input shift register 1/Q7: R1.2
- new net Input shift register 1//PL: J1.8 (IN_PL), J11.8 (Pin_8)
- new net Input shift register 4/DS: J11.4 (Pin_4)
- no-connect marks 0 -> 2
Other:
- added sheet Input shift register 1 (Input_Shift_Register.kicad_sch)
- added sheet Input shift register 2 (Input_Shift_Register.kicad_sch)
- added sheet Input shift register 3 (Input_Shift_Register.kicad_sch)
- added sheet Input shift register 4 (Input_Shift_Register.kicad_sch)

Commit message: wip
Parts:
- added J8: Screw terminal 5V GND Out, symbol Connector:Screw_Terminal_01x02
- added R2, R3: 4.7k, symbol Device:R_Small
- added R4: 47, symbol Device:R_Small
Connections:
- net +5V: now also J8.2 (Pin_2), R2.1, R3.1
- net GND: now also J8.1 (Pin_1)
- net at J1.10 (IOX_INT), J11.10 (Pin_10): now also R4.1; no longer U2.20 (INTA)
- net at J1.12 (I2C_SCL), J11.12 (Pin_12), U2.12 (SCK): now also R3.2
- net at J1.14 (I2C_SDA), J11.14 (Pin_14), U2.13 (SDA): now also R2.2
- new net: R4.2, U2.20 (INTA)

Commit message: wip
Parts:
- added C5: 100nF, symbol Device:C_Small
- added R5: 1k, symbol Device:R_Small
Connections:
- net GND: now also C5.2
- net at J1., J1.24 (ANA_DA): now also C5.1, R5.1; no longer U5.3 (A)
- new net: R5.2, U5.3 (A)
