File: PCBs/Right_Main/Input_Shift_Register.kicad_sch (KiCad schematic)
At the start: 4 parts, among them J4 Screw_Terminal_01x08, U4 74HC165

Commit message: wip
Parts:
- renumbered C5 to C3, J4 to J2, RN1 to RN3, U4 to U2

Commit message: wip
Parts:
- renumbered C3 to C4, J2 to J10, RN3 to RN1, U2 to U4
Changed lines of the file:
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@@
 		(on_board yes)
 		(dnp no)
-		(property "Reference" "J2"
+		(property "Reference" "J10"
 			(at 100.33 88.8999 0)
 			(effects
@@
 			(project ""
 				(path "/70ceab5e-e31b-4508-a755-c321a835a8c9/06890bf6-dd23-4e88-9f1e-ae85625d1e22"
-					(reference "J2")
+					(reference "J12")
 					(unit 1)
 				)
 				(path "/70ceab5e-e31b-4508-a755-c321a835a8c9/1118328f-a1b2-4dcf-b1c5-36c97ae5f908"
-					(reference "J2")
+					(reference "J10")
 					(unit 1)
 				)
 				(path "/70ceab5e-e31b-4508-a755-c321a835a8c9/689e04ea-9ab8-44cb-ac25-fd1df69ea6ca"
-					(reference "J12")
+					(reference "J14")
 					(unit 1)
 				)
 				(path "/70ceab5e-e31b-4508-a755-c321a835a8c9/69476812-841e-42e1-9ee1-30f93f6ede61"
-					(reference "J2")
+					(reference "J11")
 					(unit 1)
 				)
 				(path "/70ceab5e-e31b-4508-a755-c321a835a8c9/b184a816-d02f-4ef9-897c-d31b5b062636"
-					(reference "J2")
+					(reference "J13")
 					(unit 1)
 				)
 				(path "/70ceab5e-e31b-4508-a755-c321a835a8c9/ffdc2058-e5d3-4693-94cd-ce1a8b4b8c8e"
-					(reference "J1")
+					(reference "J15")
 					(unit 1)
 				)
@@
 		(dnp no)
 		(fields_autoplaced yes)
-		(property "Reference" "#PWR011"
+		(property "Reference" "#PWR029"
 			(at 160.02 57.15 0)
 			(effects
@@
 			(project ""
 				(path "/70ceab5e-e31b-4508-a755-c321a835a8c9/06890bf6-dd23-4e88-9f1e-ae85625d1e22"
-					(reference "#PWR011")
+					(reference "#PWR039")
 					(unit 1)
 				)
 				(path "/70ceab5e-e31b-4508-a755-c321a835a8c9/1118328f-a1b2-4dcf-b1c5-36c97ae5f908"
-					(reference "#PWR011")
+					(reference "#PWR029")
 					(unit 1)
 				)
 				(path "/70ceab5e-e31b-4508-a755-c321a835a8c9/689e04ea-9ab8-44cb-ac25-fd1df69ea6ca"
-					(reference "#PWR043")
+					(reference "#PWR049")
 					(unit 1)
 				)
 				(path "/70ceab5e-e31b-4508-a755-c321a835a8c9/69476812-841e-42e1-9ee1-30f93f6ede61"
-					(reference "#PWR011")
+					(reference "#PWR034")
 					(unit 1)
 				)
 				(path "/70ceab5e-e31b-4508-a755-c321a835a8c9/b184a816-d02f-4ef9-897c-d31b5b062636"
-					(reference "#PWR011")
+					(reference "#PWR044")
 					(unit 1)
 				)
 				(path "/70ceab5e-e31b-4508-a755-c321a835a8c9/ffdc2058-e5d3-4693-94cd-ce1a8b4b8c8e"
-					(reference "#PWR04")
+					(reference "#PWR054")
 					(unit 1)
 				)
@@
 		(dnp no)
 		(fields_autoplaced yes)
-		(property "Reference" "#PWR07"
+		(property "Reference" "#PWR026"
 			(at 116.84 62.23 0)
 			(effects
@@
 			(project ""
 				(path "/70ceab5e-e31b-4508-a755-c321a835a8c9/06890bf6-dd23-4e88-9f1e-ae85625d1e22"
-					(reference "#PWR07")
+					(reference "#PWR036")
 					(unit 1)
 				)
 				(path "/70ceab5e-e31b-4508-a755-c321a835a8c9/1118328f-a1b2-4dcf-b1c5-36c97ae5f908"
-					(reference "#PWR07")
+					(reference "#PWR026")
 					(unit 1)
 				)
 				(path "/70ceab5e-e31b-4508-a755-c321a835a8c9/689e04ea-9ab8-44cb-ac25-fd1df69ea6ca"
-					(reference "#PWR039")
+					(reference "#PWR046")
 					(unit 1)
 				)
 				(path "/70ceab5e-e31b-4508-a755-c321a835a8c9/69476812-841e-42e1-9ee1-30f93f6ede61"
-					(reference "#PWR07")
+					(reference "#PWR031")
 					(unit 1)
 				)
 				(path "/70ceab5e-e31b-4508-a755-c321a835a8c9/b184a816-d02f-4ef9-897c-d31b5b062636"
-					(reference "#PWR07")
+					(reference "#PWR041")
 					(unit 1)
 				)
 				(path "/70ceab5e-e31b-4508-a755-c321a835a8c9/ffdc2058-e5d3-4693-94cd-ce1a8b4b8c8e"
-					(reference "#PWR01")
+					(reference "#PWR051")
 					(unit 1)
 				)
@@
 		(dnp no)
 		(fields_autoplaced yes)
-		(property "Reference" "C3"
+		(property "Reference" "C4"
 			(at 162.56 64.7762 0)
 			(effects
@@
 			(project ""
 				(path "/70ceab5e-e31b-4508-a755-c321a835a8c9/06890bf6-dd23-4e88-9f1e-ae85625d1e22"
-					(reference "C3")
+					(reference "C6")
 					(unit 1)
 				)
 				(path "/70ceab5e-e31b-4508-a755-c321a835a8c9/1118328f-a1b2-4dcf-b1c5-36c97ae5f908"
-					(reference "C3")
+					(reference "C4")
 					(unit 1)
 				)
@@
 				)
 				(path "/70ceab5e-e31b-4508-a755-c321a835a8c9/69476812-841e-42e1-9ee1-30f93f6ede61"
-					(reference "C3")
+					(reference "C5")
 					(unit 1)
 				)
 				(path "/70ceab5e-e31b-4508-a755-c321a835a8c9/b184a816-d02f-4ef9-897c-d31b5b062636"
-					(reference "C3")
+					(reference "C7")
 					(unit 1)
 				)
 				(path "/70ceab5e-e31b-4508-a755-c321a835a8c9/ffdc2058-e5d3-4693-94cd-ce1a8b4b8c8e"
-					(reference "C2")
+					(reference "C9")
 					(unit 1)
 				)
@@
 		(dnp no)
 		(fields_autoplaced yes)
-		(property "Reference" "#PWR012"
+		(property "Reference" "#PWR030"
 			(at 160.02 125.73 0)
 			(effects
@@
 			(project ""
 				(path "/70ceab5e-e31b-4508-a755-c321a835a8c9/06890bf6-dd23-4e88-9f1e-ae85625d1e22"
-					(reference "#PWR012")
+					(reference "#PWR040")
 					(unit 1)
 				)
 				(path "/70ceab5e-e31b-4508-a755-c321a835a8c9/1118328f-a1b2-4dcf-b1c5-36c97ae5f908"
-					(reference "#PWR012")
+					(reference "#PWR030")
 					(unit 1)
 				)
 				(path "/70ceab5e-e31b-4508-a755-c321a835a8c9/689e04ea-9ab8-44cb-ac25-fd1df69ea6ca"
-					(reference "#PWR044")
+					(reference "#PWR050")
 					(unit 1)
 				)
 				(path "/70ceab5e-e31b-4508-a755-c321a835a8c9/69476812-841e-42e1-9ee1-30f93f6ede61"
-					(reference "#PWR012")
+					(reference "#PWR035")
 					(unit 1)
 				)
 				(path "/70ceab5e-e31b-4508-a755-c321a835a8c9/b184a816-d02f-4ef9-897c-d31b5b062636"
-					(reference "#PWR012")
+					(reference "#PWR045")
 					(unit 1)
 				)
 				(path "/70ceab5e-e31b-4508-a755-c321a835a8c9/ffdc2058-e5d3-4693-94cd-ce1a8b4b8c8e"
-					(reference "#PWR05")
+					(reference "#PWR055")
 					(unit 1)
 				)
@@
 		(dnp no)
 		(fields_autoplaced yes)
-		(property "Reference" "#PWR09"
+		(property "Reference" "#PWR028"
 			(at 162.56 69.85 0)
 			(effects
@@
 			(project ""
 				(path "/70ceab5e-e31b-4508-a755-c321a835a8c9/06890bf6-dd23-4e88-9f1e-ae85625d1e22"
-					(reference "#PWR09")
+					(reference "#PWR038")
 					(unit 1)
 				)
 				(path "/70ceab5e-e31b-4508-a755-c321a835a8c9/1118328f-a1b2-4dcf-b1c5-36c97ae5f908"
-					(reference "#PWR09")
+					(reference "#PWR028")
 					(unit 1)
 				)
 				(path "/70ceab5e-e31b-4508-a755-c321a835a8c9/689e04ea-9ab8-44cb-ac25-fd1df69ea6ca"
-					(reference "#PWR042")
+					(reference "#PWR048")
 					(unit 1)
 				)
 				(path "/70ceab5e-e31b-4508-a755-c321a835a8c9/69476812-841e-42e1-9ee1-30f93f6ede61"
-					(reference "#PWR09")
+					(reference "#PWR033")
 					(unit 1)
 				)
 				(path "/70ceab5e-e31b-4508-a755-c321a835a8c9/b184a816-d02f-4ef9-897c-d31b5b062636"
-					(reference "#PWR09")
+					(reference "#PWR043")
 					(unit 1)
 				)
 				(path "/70ceab5e-e31b-4508-a755-c321a835a8c9/ffdc2058-e5d3-4693-94cd-ce1a8b4b8c8e"
-					(reference "#PWR03")
+					(reference "#PWR053")
 					(unit 1)
 				)
@@
 		(dnp no)
 		(fields_autoplaced yes)
-		(property "Reference" "RN3"
+		(property "Reference" "RN1"
 			(at 137.16 62.4839 0)
 			(effects
@@
 				)
 				(path "/70ceab5e-e31b-4508-a755-c321a835a8c9/1118328f-a1b2-4dcf-b1c5-36c97ae5f908"
-					(reference "RN3")
+					(reference "RN1")
 					(unit 1)
 				)
@@
 				)
 				(path "/70ceab5e-e31b-4508-a755-c321a835a8c9/69476812-841e-42e1-9ee1-30f93f6ede61"
-					(reference "RN3")
+					(reference "RN2")
 					(unit 1)
 				)
 				(path "/70ceab5e-e31b-4508-a755-c321a835a8c9/b184a816-d02f-4ef9-897c-d31b5b062636"
-					(reference "RN3")
+					(reference "RN4")
 					(unit 1)
 				)
 				(path "/70ceab5e-e31b-4508-a755-c321a835a8c9/ffdc2058-e5d3-4693-94cd-ce1a8b4b8c8e"
-					(reference "RN1")
+					(reference "RN6")
 					(unit 1)
 				)
@@
 		(dnp no)
 		(fields_autoplaced yes)
-		(property "Reference" "#PWR08"
+		(property "Reference" "#PWR027"
 			(at 140.97 111.76 0)
 			(effects
@@
 			(project ""
 				(path "/70ceab5e-e31b-4508-a755-c321a835a8c9/06890bf6-dd23-4e88-9f1e-ae85625d1e22"
-					(reference "#PWR08")
+					(reference "#PWR037")
 					(unit 1)
 				)
 				(path "/70ceab5e-e31b-4508-a755-c321a835a8c9/1118328f-a1b2-4dcf-b1c5-36c97ae5f908"
-					(reference "#PWR08")
+					(reference "#PWR027")
 					(unit 1)
 				)
 				(path "/70ceab5e-e31b-4508-a755-c321a835a8c9/689e04ea-9ab8-44cb-ac25-fd1df69ea6ca"
-					(reference "#PWR041")
+					(reference "#PWR047")
 					(unit 1)
 				)
 				(path "/70ceab5e-e31b-4508-a755-c321a835a8c9/69476812-841e-42e1-9ee1-30f93f6ede61"
-					(reference "#PWR08")
+					(reference "#PWR032")
 					(unit 1)
 				)
 				(path "/70ceab5e-e31b-4508-a755-c321a835a8c9/b184a816-d02f-4ef9-897c-d31b5b062636"
-					(reference "#PWR08")
+					(reference "#PWR042")
 					(unit 1)
 				)
 				(path "/70ceab5e-e31b-4508-a755-c321a835a8c9/ffdc2058-e5d3-4693-94cd-ce1a8b4b8c8e"
-					(reference "#PWR02")
+					(reference "#PWR052")
 					(unit 1)
 				)
@@
 		(on_board yes)
 		(dnp no)
-		(property "Reference" "U2"
+		(property "Reference" "U4"
 			(at 162.1633 71.12 0)
 			(effects
@@
 			(project ""
 				(path "/70ceab5e-e31b-4508-a755-c321a835a8c9/06890bf6-dd23-4e88-9f1e-ae85625d1e22"
-					(reference "U2")
+					(reference "U6")
 					(unit 1)
 				)
 				(path "/70ceab5e-e31b-4508-a755-c321a835a8c9/1118328f-a1b2-4dcf-b1c5-36c97ae5f908"
-					(reference "U2")
+					(reference "U4")
 					(unit 1)
 				)
@@
 				)
 				(path "/70ceab5e-e31b-4508-a755-c321a835a8c9/69476812-841e-42e1-9ee1-30f93f6ede61"
-					(reference "U2")
+					(reference "U5")
 					(unit 1)
 				)
 				(path "/70ceab5e-e31b-4508-a755-c321a835a8c9/b184a816-d02f-4ef9-897c-d31b5b062636"
-					(reference "U2")
+					(reference "U7")
 					(unit 1)
 				)
 				(path "/70ceab5e-e31b-4508-a755-c321a835a8c9/ffdc2058-e5d3-4693-94cd-ce1a8b4b8c8e"
-					(reference "U1")
-					(unit 1)
-				)
+					(reference "U9")
+					(unit 1)
+				)
