File: PCBs/Right_Main/Right_Main.kicad_sch (KiCad schematic)
At the start: 23 parts, among them J1 Future expansion, J16 Conn_RJ45_Right_To_Left, J2 Screw terminal 5V GND Out, J3 Encoder inputs B, J4 Encoder inputs A, J5 Analog inputs, J6 Future expansion, J7 Conn_Right_Keypad, J8 Rotary switchs' pin 1, J9 Analog inputs, U1 MCP23017_SP, U10 MAX485E, U2 ULN2003A, U3 74HC4051

Commit message: stuff
Connections:
- net GND: now also J7.11 (GND_6), J7.13 (GND_7), J7.15 (GND_8)
- net at A1.D10: now also J7.14 (ROW_2)
- net at U2.1 (I1), U2.2 (I2), U2.3 (I3)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: now also A1.D12; no longer A1.D11
- net at A1.D9: now also J7.12 (ROW_1)
- new net: A1.D11, J7.16 (ROW_3)
- no-connect marks 8 -> 9
Other:
- note removed: "IN_DFM (data from master) is probably not needed anymore as this shift register chain will not be chained with the left side"

Commit message: right main pcb draft
Parts:
- removed C3: 100nF, symbol Device:C_Small
- removed J1, J6: Future expansion, symbol Connector_Generic:Conn_02x13_Odd_Even
- removed J9: Analog inputs, symbol Connector:Screw_Terminal_01x08
- removed R4, R5: 100, symbol Device:R_Small
- removed U3: 74HC4051, symbol 74xx:74HC4051
- C1, C2: footprint (none) -> Capacitor_THT:C_Disc_D5.0mm_W2.5mm_P2.50mm
- J16: footprint (none) -> Connector_RJ:RJ45_Amphenol_54602-x08_Horizontal
- J2: footprint (none) -> TerminalBlock_Phoenix:TerminalBlock_Phoenix_MPT-0,5-2-2.54_1x02_P2.54mm_Horizontal
- J3, J4: footprint (none) -> TerminalBlock_Phoenix:TerminalBlock_Phoenix_MPT-0,5-8-2.54_1x08_P2.54mm_Horizontal
- J5: footprint (none) -> TerminalBlock_Phoenix:TerminalBlock_Phoenix_MPT-0,5-6-2.54_1x06_P2.54mm_Horizontal
- J7: footprint (none) -> Connector_IDC:IDC-Header_2x08_P2.54mm_Vertical
- J8: footprint (none) -> TerminalBlock_Phoenix:TerminalBlock_Phoenix_MPT-0,5-7-2.54_1x07_P2.54mm_Horizontal
- R1, R2, R3: footprint (none) -> Resistor_THT:R_Axial_DIN0207_L6.3mm_D2.5mm_P7.62mm_Horizontal
- U10: footprint Package_SO:SOIC-8_3.9x4.9mm_P1.27mm -> Package_DIP:DIP-8_W7.62mm
- U2: footprint (none) -> Package_DIP:DIP-16_W7.62mm
Connections:
- net Input register 1/CP: now also A1.D5
- net Input register 1//PL: now also A1.D6
- net at J4.1 (Pin_1): now also U1.28 (GPA7); no longer U1.21 (GPA0)
- net at J4.2 (Pin_2): now also U1.27 (GPA6); no longer U1.22 (GPA1)
- net at J4.3 (Pin_3): now also U1.26 (GPA5); no longer U1.23 (GPA2)
- net at J4.4 (Pin_4): now also U1.25 (GPA4); no longer U1.24 (GPA3)
- net at J4.5 (Pin_5): now also U1.24 (GPA3); no longer U1.25 (GPA4)
- net at J4.6 (Pin_6): now also U1.23 (GPA2); no longer U1.26 (GPA5)
- net at J4.7 (Pin_7): now also U1.22 (GPA1); no longer U1.27 (GPA6)
- net at J4.8 (Pin_8): now also U1.21 (GPA0); no longer U1.28 (GPA7)
- net at J8.1 (Pin_1): now also U2.10 (O7); no longer U2.16 (O1)
- net at J8.2 (Pin_2): now also U2.11 (O6); no longer U2.15 (O2)
- net at J8.3 (Pin_3): now also U2.12 (O5); no longer U2.14 (O3)
- net at J8.5 (Pin_5): now also U2.14 (O3); no longer U2.12 (O5)
- net at J8.6 (Pin_6): now also U2.15 (O2); no longer U2.11 (O6)
- net at J8.7 (Pin_7): now also U2.16 (O1); no longer U2.10 (O7)
- no-connect marks 9 -> 8
Other:
- note removed: "Not needed. Connected directly to the Arduino instead"
- note removed: "or just through-holes by the arduino/relevant ICs?"
- moved on the sheet: J16, J2, U10

Commit message: tweaks
Parts:
- removed J2: Screw terminal 5V GND Out, TerminalBlock_Phoenix:TerminalBlock_Phoenix_MPT-0,5-2-2.54_1x02_P2.54mm_Horizontal, symbol Connector:Screw_Terminal_01x02
- added R4, R5, R6: 470, Resistor_THT:R_Axial_DIN0207_L6.3mm_D2.5mm_P7.62mm_Horizontal, symbol Device:R_Small
Connections:
- net at J7.12 (ROW_1): now also R4.2; no longer A1.D9
- net at J7.14 (ROW_2): now also R5.2; no longer A1.D10
- net at A1.D11: now also R6.1; no longer J7.16 (ROW_3)
- new net: J7.16 (ROW_3), R6.2
- new net: A1.D10, R5.1
- new net: A1.D9, R4.1
