File: PCBs/Right_Main/Right_Main.kicad_sch (KiCad schematic)
At the start: 18 parts, among them J16 Conn_RJ45_Right_To_Left, J3 Encoder inputs B, J4 Encoder inputs A, J5 Analog inputs, J7 Conn_Right_Keypad, J8 Rotary switchs' pin 1, U1 MCP23017_SP, U10 MAX485E, U2 ULN2003A

Commit message: wip
Parts:
- added J1: Screw_Terminal_01x10, TerminalBlock_Phoenix:TerminalBlock_Phoenix_MPT-0,5-10-2.54_1x10_P2.54mm_Horizontal, symbol Connector:Screw_Terminal_01x10
Connections:
- net GND: now also J1.1 (Pin_1), J1.10 (Pin_10), J1.2 (Pin_2), J1.3 (Pin_3), J1.4 (Pin_4), J1.5 (Pin_5), J1.6 (Pin_6), J1.7 (Pin_7), J1.8 (Pin_8), J1.9 (Pin_9)
- no-connect marks 8 -> 7

Commit message: stuff
Parts:
- removed J1: Screw_Terminal_01x10, TerminalBlock_Phoenix:TerminalBlock_Phoenix_MPT-0,5-10-2.54_1x10_P2.54mm_Horizontal, symbol Connector:Screw_Terminal_01x10
- added J1: +5V and GND, TerminalBlock_Phoenix:TerminalBlock_Phoenix_MPT-0,5-8-2.54_1x08_P2.54mm_Horizontal, symbol Connector:Screw_Terminal_01x08
Connections:
- net +5V: now also J1.1 (Pin_1), J1.2 (Pin_2), J1.3 (Pin_3), J1.4 (Pin_4)
- net GND: now also J1.5 (Pin_5), J1.6 (Pin_6), J1.7 (Pin_7), J1.8 (Pin_8)

Commit message: stuff
Other:
- note added: "TODO: ESD protection? TVS diodes? For both RS485 and power"
Changed lines of the file:
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@@
 	(generator_version "10.0")
 	(paper "A4")
+	(text "TODO: ESD protection? TVS diodes? For both RS485 and power"
+		(exclude_from_sim no)
+		(at 49.53 53.34 0)
+		(effects
+			(font
+				(size 1.27 1.27)
+				(thickness 0.254)
+				(bold yes)
+				(color 255 0 0 1)
+			)
+		)
+	)
 	(text "TODO: termination resistors?"
 		(exclude_from_sim no)
