File: PCBs/Right_Main/Right_Main.kicad_pcb (KiCad board)
At the start: 2 copper layers, 221 x 111.8 mm, 40 parts, among them J10 Screw_Terminal_01x08, J11 Screw_Terminal_01x08, J12 Screw_Terminal_01x08, J13 Screw_Terminal_01x08, J14 Screw_Terminal_01x08, J15 Screw_Terminal_01x08, J16 Conn_RJ45_Right_To_Left, J2 Screw terminal 5V GND Out, J3 Encoder inputs B, J4 Encoder inputs A, J5 Analog inputs, J7 Conn_Right_Keypad, J8 Rotary switchs' pin 1, U1 MCP23017_SP, U10 MAX485E, U2 ULN2003A, U4 74HC165, U5 74HC165, U6 74HC165, U7 74HC165, U8 74HC165, U9 74HC165

Commit message: right main pcb draft 2 wip
Parts:
- moved C6 44.9 mm to (179.7, 99.7)
- moved U10 44.9 mm to (181.6, 78.7)
- moved U2 44.9 mm to (253.4, 99.1)
- moved U4 44.9 mm to (227.3, 95.2)
- moved C7 44.9 mm to (154.3, 99.7)
- moved C8 44.9 mm to (128.9, 99.7)
- moved J13 44.9 mm to (134.0, 111.8)
- moved J7 44.9 mm to (72.4, 92.7)
- moved RN1 44.9 mm to (229.9, 106.0)
- moved U1 44.9 mm to (214.0, 90.2)
- moved U8 44.9 mm to (125.7, 95.2)
- moved U9 44.9 mm to (100.3, 95.2)
- moved C4 44.9 mm to (230.5, 99.7)
- moved C9 44.9 mm to (103.5, 99.7)
- moved J16 44.9 mm to (204.9, 82.6)
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Routing:
- net +5V: track 405.0 -> 0.00 mm
- net Net-(U10-DE): track 74.3 -> 60.3 mm, vias 0 -> 1
- net Net-(A1-D1/TX): track 45.6 -> 34.5 mm
- net /Input register 1//PL: track 196.4 -> 187.3 mm, vias 7 -> 2
- net /Input register 1/CP: track 191.8 -> 183.5 mm
- net Net-(A1-D0/RX): track 41.2 -> 33.9 mm, vias 0 -> 1
- net Net-(J16-485_B): track 22.6 -> 16.0 mm
- net Net-(A1-D7_INT4): track 126.8 -> 121.9 mm, vias 5 -> 4
- net Net-(J15-Pin_7): track 25.1 -> 29.7 mm, vias 2 -> 0
- net Net-(J13-Pin_7): track 25.1 -> 29.7 mm, vias 2 -> 0
- net Net-(J14-Pin_7): track 25.1 -> 29.7 mm, vias 2 -> 0
- net Net-(J11-Pin_7): track 25.1 -> 29.7 mm, vias 2 -> 0
- net Net-(J10-Pin_7): track 25.1 -> 29.7 mm, vias 2 -> 0
- net Net-(J12-Pin_7): track 25.1 -> 29.7 mm, vias 2 -> 0
- net Net-(A1-D2/SDA): track 114.2 -> 118.4 mm, vias 5 -> 1
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- added copper zone on In2.Cu, net +5V
- added copper zone on In1.Cu, net GND
- removed copper zone on B.Cu, net GND
Other:
- board size 221 x 111.8 mm -> 195.6 x 55.9 mm
- copper layers 2 -> 4

Commit message: tweaks
Parts:
- removed J2: Screw terminal 5V GND Out, TerminalBlock_Phoenix:TerminalBlock_Phoenix_MPT-0,5-2-2.54_1x02_P2.54mm_Horizontal
- added R4: 470, Resistor_THT:R_Axial_DIN0207_L6.3mm_D2.5mm_P7.62mm_Horizontal, F.Cu at (108.6, 66.0)
- added R5: 470, Resistor_THT:R_Axial_DIN0207_L6.3mm_D2.5mm_P7.62mm_Horizontal, F.Cu at (108.6, 69.8)
- added R6: 470, Resistor_THT:R_Axial_DIN0207_L6.3mm_D2.5mm_P7.62mm_Horizontal, F.Cu at (108.6, 73.7)
Connections:
- A1 pad D10: Net-(J7-ROW_2) -> Net-(A1-PadD10)
- A1 pad D11: Net-(J7-ROW_3) -> Net-(A1-PadD11)
- A1 pad D9: Net-(J7-ROW_1) -> Net-(A1-PadD9)
Routing:
- net Net-(J7-ROW_1): track 70.0 -> 50.2 mm
- net Net-(A1-PadD9): track 0.00 -> 19.0 mm
- net Net-(J7-ROW_2): track 68.7 -> 50.4 mm
- net Net-(J7-ROW_3): track 67.5 -> 50.6 mm
- net Net-(A1-PadD10): track 0.00 -> 14.9 mm
- net Net-(A1-PadD11): track 0.00 -> 11.8 mm

Commit message: wip
Parts:
- added J1: Screw_Terminal_01x10, TerminalBlock_Phoenix:TerminalBlock_Phoenix_MPT-0,5-10-2.54_1x10_P2.54mm_Horizontal, F.Cu at (183.5, 71.1)
- moved J16 126.5 mm to (78.7, 73.7)
- moved U10 89.0 mm to (92.7, 74.9), turned to 180 degrees
- moved R6 24.4 mm to (89.5, 88.9)
- moved R4 23.0 mm to (111.1, 88.9)
- moved R5 20.8 mm to (100.3, 88.9)
Routing:
- net Net-(A1-D1/TX): track 34.5 -> 62.3 mm
- net Net-(J7-ROW_3): track 50.6 -> 24.5 mm, vias 0 -> 1
- net Net-(A1-D0/RX): track 33.9 -> 59.3 mm
- net Net-(A1-PadD11): track 11.8 -> 36.2 mm
- net Net-(U10-DE): track 60.3 -> 37.4 mm, vias 1 -> 0
- net Net-(J7-ROW_2): track 50.4 -> 32.0 mm
- net Net-(A1-PadD10): track 14.9 -> 27.9 mm
- net Net-(J16-485_A): track 17.3 -> 7.92 mm
- net Net-(J7-ROW_1): track 50.2 -> 41.0 mm, vias 0 -> 1
- net Net-(J16-485_B): track 16.0 -> 9.19 mm
- net Net-(A1-D7_INT4): track 121.9 -> 118.8 mm, vias 4 -> 3
- net Net-(A1-PadD9): track 19.0 -> 20.8 mm

Commit message: stuff
Parts:
- J1: value Screw_Terminal_01x10 -> +5V and GND; footprint TerminalBlock_Phoenix:TerminalBlock_Phoenix_MPT-0,5-10-2.54_1x10_P2.54mm_Horizontal -> TerminalBlock_Phoenix:TerminalBlock_Phoenix_MPT-0,5-8-2.54_1x08_P2.54mm_Horizontal
- moved J1 2.55 mm to (186.1, 70.9)
Connections:
- J1 pad 1: GND -> +5V
- J1 pad 2: GND -> +5V
- J1 pad 3: GND -> +5V
- J1 pad 4: GND -> +5V
Other:
- board text added: "+5"
- board text added: "GND"

Commit message: stuff
Connections:
- J3 pad 1: Net-(J3-Pin_1) -> Net-(J3-Pin_8)
- J3 pad 2: Net-(J3-Pin_2) -> Net-(J3-Pin_7)
- J3 pad 3: Net-(J3-Pin_3) -> Net-(J3-Pin_6)
- J3 pad 4: Net-(J3-Pin_4) -> Net-(J3-Pin_5)
- J3 pad 5: Net-(J3-Pin_5) -> Net-(J3-Pin_4)
- J3 pad 6: Net-(J3-Pin_6) -> Net-(J3-Pin_3)
- J3 pad 7: Net-(J3-Pin_7) -> Net-(J3-Pin_2)
- J3 pad 8: Net-(J3-Pin_8) -> Net-(J3-Pin_1)
Routing:
- net Net-(J3-Pin_8): track 29.6 -> 61.0 mm
- net Net-(J3-Pin_7): track 29.6 -> 59.5 mm
- net Net-(J3-Pin_6): track 29.6 -> 58.1 mm
- net Net-(J3-Pin_5): track 29.6 -> 56.6 mm
- net Net-(J3-Pin_4): track 29.6 -> 55.1 mm
- net Net-(J3-Pin_3): track 29.6 -> 53.6 mm
- net Net-(J3-Pin_2): track 29.6 -> 52.1 mm
- net Net-(J3-Pin_1): track 29.6 -> 47.4 mm
- added copper zone on B.Cu, net GND
- added copper zone on F.Cu, net GND
