File: PCBs/Right_Keypad/Right_Keypad.kicad_sch (KiCad schematic)
At the start: 63 parts, among them J1 Conn_Right_Keypad, Q1 NPN, Q2 NPN, Q3 NPN, SW1 SW_Push, SW10 SW_Push, SW11 SW_Push, SW12 SW_Push, SW13 SW_Push, SW14 SW_Push, SW15 SW_Push, SW16 SW_Push, SW17 SW_Push, SW18 SW_Push, SW19 SW_Push, SW2 SW_Push, SW20 SW_Push, SW21 SW_Push, SW22 SW_Push, SW23 SW_Push, SW24 SW_Push, SW3 SW_Push, SW4 SW_Push, SW5 SW_Push, SW6 SW_Push, SW7 SW_Push, SW8 SW_Push, SW9 SW_Push, U1 74HC165

Commit message: keypad 3v3, before removing transistors
Connections:
- net +5V renamed +3V3

Commit message: stuff
Parts:
- removed Q1, Q2, Q3: NPN, Package_TO_SOT_THT:TO-92_Inline, symbol Transistor_BJT:Q_NPN_CBE
- removed R2, R3, R4: 10k, Resistor_THT:R_Axial_DIN0207_L6.3mm_D2.5mm_P7.62mm_Horizontal, symbol Device:R_Small
Connections:
- net at SW10.1, SW11.1, SW12.1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: now also J1.14 (ROW_2)
- net at SW1.1, SW2.1, SW3.1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: now also J1.12 (ROW_1)
- net at SW17.1, SW18.1, SW19.1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: now also J1.16 (ROW_3)
