File: PCBs/Right_Keypad/Right_Keypad.kicad_sch (KiCad schematic)
At the start: 57 parts, among them J1 Conn_Right_Keypad, SW1 SW_Push, SW10 SW_Push, SW11 SW_Push, SW12 SW_Push, SW13 SW_Push, SW14 SW_Push, SW15 SW_Push, SW16 SW_Push, SW17 SW_Push, SW18 SW_Push, SW19 SW_Push, SW2 SW_Push, SW20 SW_Push, SW21 SW_Push, SW22 SW_Push, SW23 SW_Push, SW24 SW_Push, SW3 SW_Push, SW4 SW_Push, SW5 SW_Push, SW6 SW_Push, SW7 SW_Push, SW8 SW_Push, SW9 SW_Push, U1 74HC165

Commit message: stuff
Changed lines of the file:
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@@
 	(generator_version "10.0")
 	(paper "A4")
-	(text_box "A while after designing this: I think the transistors had something to do with the 3 row lines also being used as address lines for the analog multiplexers (which I removed later) (and then added again). Not sure. Not gonna remove them now."
-		(exclude_from_sim no)
-		(at 58.42 147.32 0)
-		(size 29.21 22.86)
-		(margins 0.9525 0.9525 0.9525 0.9525)
-		(stroke
-			(width 0)
-			(type solid)
-		)
-		(fill
-			(type none)
-		)
-		(effects
-			(font
-				(size 1.27 1.27)
-			)
-			(justify left top)
-		)
-	)
 	(junction
 		(at 121.92 111.76)

Commit message: Fixed issues identified by Claude - batch 4
Parts:
- D1, D10, D11, D12, D13, D14, D15, D16, D17, D18, D19, D2, D20, D21, D22, D23, D24, D3, D4, D5, D6, D7, D8, D9: value D -> D_Schottky; footprint Diode_SMD:D_SOD-123 -> Diode_SMD:D_SOD-323_HandSoldering; symbol Device:D -> Device:D_Schottky

Commit message: Fixed issues identified by Claude - batch 5 - done
Parts:
- D1, D10, D11, D12, D13, D14, D15, D16, D17, D18, D19, D2, D20, D21, D22, D23, D24, D3, D4, D5, D6, D7, D8, D9: value D_Schottky -> SD103AWS
Changed lines of the file:
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@@
 			)
 		)
-		(property "Value" "D_Schottky"
+		(property "Value" "SD103AWS"
 			(at 194.31 149.86 0)
 			(hide yes)
@@
 			)
 		)
-		(property "Value" "D_Schottky"
+		(property "Value" "SD103AWS"
 			(at 175.26 149.86 0)
 			(hide yes)
@@
 			)
 		)
-		(property "Value" "D_Schottky"
+		(property "Value" "SD103AWS"
 			(at 156.21 149.86 0)
 			(hide yes)
@@
 			)
 		)
-		(property "Value" "D_Schottky"
+		(property "Value" "SD103AWS"
 			(at 251.46 132.08 0)
 			(hide yes)
@@
 			)
 		)
-		(property "Value" "D_Schottky"
+		(property "Value" "SD103AWS"
 			(at 213.36 114.3 0)
 			(hide yes)
@@
 			)
 		)
-		(property "Value" "D_Schottky"
+		(property "Value" "SD103AWS"
 			(at 232.41 132.08 0)
 			(hide yes)
@@
 			)
 		)
-		(property "Value" "D_Schottky"
+		(property "Value" "SD103AWS"
 			(at 213.36 149.86 0)
 			(hide yes)
@@
 			)
 		)
-		(property "Value" "D_Schottky"
+		(property "Value" "SD103AWS"
 			(at 232.41 114.3 0)
 			(hide yes)
@@
 			)
 		)
-		(property "Value" "D_Schottky"
+		(property "Value" "SD103AWS"
 			(at 175.26 114.3 0)
 			(hide yes)
@@
 			)
 		)
-		(property "Value" "D_Schottky"
+		(property "Value" "SD103AWS"
 			(at 137.16 132.08 0)
 			(hide yes)
@@
 			)
 		)
-		(property "Value" "D_Schottky"
+		(property "Value" "SD103AWS"
 			(at 213.36 132.08 0)
 			(hide yes)
@@
 			)
 		)
-		(property "Value" "D_Schottky"
+		(property "Value" "SD103AWS"
 			(at 137.16 114.3 0)
 			(hide yes)
@@
 			)
 		)
-		(property "Value" "D_Schottky"
+		(property "Value" "SD103AWS"
 			(at 156.21 114.3 0)
 			(hide yes)
@@
 			)
 		)
-		(property "Value" "D_Schottky"
+		(property "Value" "SD103AWS"
 			(at 156.21 132.08 0)
 			(hide yes)
@@
 			)
 		)
-		(property "Value" "D_Schottky"
+		(property "Value" "SD103AWS"
 			(at 175.26 132.08 0)
 			(hide yes)
@@
 			)
 		)
-		(property "Value" "D_Schottky"
+		(property "Value" "SD103AWS"
 			(at 251.46 114.3 0)
 			(hide yes)
@@
 			)
 		)
-		(property "Value" "D_Schottky"
+		(property "Value" "SD103AWS"
 			(at 118.11 149.86 0)
 			(hide yes)
@@
 			)
 		)
-		(property "Value" "D_Schottky"
+		(property "Value" "SD103AWS"
 			(at 232.41 149.86 0)
 			(hide yes)
@@
 			)
 		)
-		(property "Value" "D_Schottky"
+		(property "Value" "SD103AWS"
 			(at 118.11 132.08 0)
 			(hide yes)
@@
 			)
 		)
-		(property "Value" "D_Schottky"
+		(property "Value" "SD103AWS"
 			(at 194.31 114.3 0)
 			(hide yes)
@@
 			)
 		)
-		(property "Value" "D_Schottky"
+		(property "Value" "SD103AWS"
 			(at 137.16 149.86 0)
 			(hide yes)
@@
 			)
 		)
-		(property "Value" "D_Schottky"
+		(property "Value" "SD103AWS"
 			(at 194.31 132.08 0)
 			(hide yes)
@@
 			)
 		)
-		(property "Value" "D_Schottky"
+		(property "Value" "SD103AWS"
 			(at 118.11 114.3 0)
 			(hide yes)
@@
 			)
 		)
-		(property "Value" "D_Schottky"
+		(property "Value" "SD103AWS"
 			(at 251.46 149.86 0)
 			(hide yes)
