File: PCBs/Right_Keypad/Right_Keypad.kicad_pcb (KiCad board)
At the start: 4 copper layers, 86.3 x 106.6 mm, 63 parts, among them J1 Conn_Right_Keypad, Q1 NPN, Q2 NPN, Q3 NPN, SW1 SW_Push, SW10 SW_Push, SW11 SW_Push, SW12 SW_Push, SW13 SW_Push, SW14 SW_Push, SW15 SW_Push, SW16 SW_Push, SW17 SW_Push, SW18 SW_Push, SW19 SW_Push, SW2 SW_Push, SW20 SW_Push, SW21 SW_Push, SW22 SW_Push, SW23 SW_Push, SW24 SW_Push, SW3 SW_Push, SW4 SW_Push, SW5 SW_Push, SW6 SW_Push, SW7 SW_Push, SW8 SW_Push, SW9 SW_Push, U1 74HC165

Commit message: right keypad ready
Routing:
- net GND: track 0.00 -> 123.7 mm, vias 0 -> 1
- net +5V: track 0.00 -> 60.2 mm, vias 0 -> 2
- removed copper zone on In2.Cu, net +5V
- removed copper zone on In1.Cu, net GND
Other:
- copper layers 4 -> 2

Commit message: right main pcb draft
Connections:
- U1 pad 10: unconnected-(U1-DS-Pad10) -> GND
Routing:
- net GND: track 123.7 -> 135.0 mm

Commit message: tweaks
Routing:
- net GND: track 135.0 -> 129.4 mm
- net Net-(Q1-C): track 205.4 -> 202.6 mm
- net Net-(Q3-C): track 152.9 -> 151.0 mm
- net Net-(Q2-C): track 168.1 -> 166.8 mm
- net Net-(U1-Q7): track 15.7 -> 14.8 mm
- net Net-(D15-A): track 112.7 -> 112.0 mm
- net Net-(D1-A): track 53.7 -> 53.1 mm
- net Net-(Q1-B): track 29.5 -> 28.9 mm
Other:
- outline, holes or cut-outs redrawn

Commit message: stuff
Parts:
- removed Q1, Q2, Q3: NPN, Package_TO_SOT_THT:TO-92_Inline
- removed R2, R3, R4: 10k, Resistor_THT:R_Axial_DIN0207_L6.3mm_D2.5mm_P7.62mm_Horizontal
Connections:
- net +5V renamed +3V3
- SW1 pad 1: Net-(Q1-C) -> Net-(J1-ROW_1)
- SW10 pad 1: Net-(Q2-C) -> Net-(J1-ROW_2)
- SW11 pad 1: Net-(Q2-C) -> Net-(J1-ROW_2)
- SW12 pad 1: Net-(Q2-C) -> Net-(J1-ROW_2)
- SW13 pad 1: Net-(Q2-C) -> Net-(J1-ROW_2)
- SW14 pad 1: Net-(Q2-C) -> Net-(J1-ROW_2)
- SW15 pad 1: Net-(Q2-C) -> Net-(J1-ROW_2)
- SW16 pad 1: Net-(Q2-C) -> Net-(J1-ROW_2)
- SW17 pad 1: Net-(Q3-C) -> Net-(J1-ROW_3)
- SW18 pad 1: Net-(Q3-C) -> Net-(J1-ROW_3)
- SW19 pad 1: Net-(Q3-C) -> Net-(J1-ROW_3)
- SW2 pad 1: Net-(Q1-C) -> Net-(J1-ROW_1)
- SW20 pad 1: Net-(Q3-C) -> Net-(J1-ROW_3)
- SW21 pad 1: Net-(Q3-C) -> Net-(J1-ROW_3)
- SW22 pad 1: Net-(Q3-C) -> Net-(J1-ROW_3)
- SW23 pad 1: Net-(Q3-C) -> Net-(J1-ROW_3)
- SW24 pad 1: Net-(Q3-C) -> Net-(J1-ROW_3)
- SW3 pad 1: Net-(Q1-C) -> Net-(J1-ROW_1)
- SW4 pad 1: Net-(Q1-C) -> Net-(J1-ROW_1)
- SW5 pad 1: Net-(Q1-C) -> Net-(J1-ROW_1)
- SW6 pad 1: Net-(Q1-C) -> Net-(J1-ROW_1)
- SW7 pad 1: Net-(Q1-C) -> Net-(J1-ROW_1)
- SW8 pad 1: Net-(Q1-C) -> Net-(J1-ROW_1)
- SW9 pad 1: Net-(Q2-C) -> Net-(J1-ROW_2)
Routing:
- net Net-(J1-ROW_1): track 25.5 -> 261.6 mm, vias 0 -> 1
- net Net-(Q1-C): track 202.6 -> 0.00 mm, vias 1 -> 0
- net Net-(J1-ROW_2): track 27.5 -> 215.6 mm, vias 0 -> 1
- net Net-(Q2-C): track 166.8 -> 0.00 mm, vias 1 -> 0
- net Net-(J1-ROW_3): track 31.6 -> 196.2 mm
- net Net-(Q3-C): track 151.0 -> 0.00 mm
- net GND: track 129.4 -> 91.0 mm, vias 1 -> 2
- net Net-(Q1-B): track 28.9 -> 0.00 mm
- net Net-(Q2-B): track 17.2 -> 0.00 mm
- net Net-(Q3-B): track 9.83 -> 0.00 mm
- net Net-(J1-IN_PL): track 57.6 -> 55.6 mm
- net Net-(J1-IN_CP): track 54.1 -> 52.5 mm
