File: PCBs/Right_Keypad/Right_Keypad.kicad_pcb (KiCad board)
At the start: 2 copper layers, 86.3 x 106.6 mm, 57 parts, among them J1 Conn_Right_Keypad, SW1 SW_Push, SW10 SW_Push, SW11 SW_Push, SW12 SW_Push, SW13 SW_Push, SW14 SW_Push, SW15 SW_Push, SW16 SW_Push, SW17 SW_Push, SW18 SW_Push, SW19 SW_Push, SW2 SW_Push, SW20 SW_Push, SW21 SW_Push, SW22 SW_Push, SW23 SW_Push, SW24 SW_Push, SW3 SW_Push, SW4 SW_Push, SW5 SW_Push, SW6 SW_Push, SW7 SW_Push, SW8 SW_Push, SW9 SW_Push, U1 74HC165

Commit message: Fix 74HC4051 enable, set pull-up values, name keypad column nets
Shared_Main:
- U2 (74HC4051) pin 6 (~E) was tied to +3V3, permanently inhibiting all
  eight analog channels. Moved to GND. The pad had no tracks on it, so
  the board change is just which plane claims it (In2 +3V3 -> In1 GND);
  all zones refilled.
- RN1-RN6 pull-up arrays had no value assigned (still reading the
  R_Network08 symbol default). Set to 10k, matching RN8. Board footprint
  value fields synced to match.
- Also includes graphical tidy-up of junction/wire placement (no netlist
  change).

Right_Keypad:
- RN1 pull-up array set to 10k, board field synced.
- U1 was using a locally modified 74HC165 whose D0-D3 pins had been moved
  (via Swap Pins) so the column rails fan out to RN1 without crossing.
  That recorded the bit-order decision in pin geometry, where nothing
  diffs it and an "Update Symbols from Library" would silently remap four
  nets. Reverted U1 to the stock 74xx:74HC165 and expressed the same
  mapping as named nets COL1-COL8 instead:

      COL1 -> D3   COL5 -> D4
      COL2 -> D2   COL6 -> D5
      COL3 -> D1   COL7 -> D6
      COL4 -> D0   COL8 -> D7

  Connectivity is unchanged - verified by diffing before/after netlists
  with net names stripped and each net's pin set sorted. No copper moved
  (363 segments, 8 vias, 57 footprints before and after); only net names
  changed on the board.

Both projects: ERC 0, DRC 0, 0 unconnected, 0 schematic parity issues.

Co-Authored-By: Claude Opus 5 <noreply@anthropic.com>
Parts:
- RN1: value R_Network08 -> 10k
Connections:
- net Net-(D1-A) renamed /COL1
- net Net-(D10-A) renamed /COL2
- net Net-(D11-A) renamed /COL3
- net Net-(D12-A) renamed /COL4
- net Net-(D13-A) renamed /COL5
- net Net-(D14-A) renamed /COL6
- net Net-(D15-A) renamed /COL7
- net Net-(D16-A) renamed /COL8
