File: PCBs/Right_Keypad/Right_Keypad.kicad_pcb (KiCad board)
At the start: 2 copper layers, 86.3 x 106.6 mm, 57 parts, among them J1 Conn_Right_Keypad, SW1 SW_Push, SW10 SW_Push, SW11 SW_Push, SW12 SW_Push, SW13 SW_Push, SW14 SW_Push, SW15 SW_Push, SW16 SW_Push, SW17 SW_Push, SW18 SW_Push, SW19 SW_Push, SW2 SW_Push, SW20 SW_Push, SW21 SW_Push, SW22 SW_Push, SW23 SW_Push, SW24 SW_Push, SW3 SW_Push, SW4 SW_Push, SW5 SW_Push, SW6 SW_Push, SW7 SW_Push, SW8 SW_Push, SW9 SW_Push, U1 74HC165

Commit message: tweaks
Routing:
- net /COL5: track 113.8 -> 112.8 mm

Commit message: Fixed issues identified by Claude - batch 2
Parts:
- moved C1 24.8 mm to (111.1, 118.7)
Routing:
- net +3V3: track 60.3 -> 76.6 mm, vias 2 -> 0
- net GND: track 91.0 -> 89.4 mm, vias 2 -> 1
Changed lines of the file:
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@@
 		(capping no)
 		(filling no)
+		(zone_defaults)
 		(pcbplotparams
 			(layerselection 0x00000000_00000000_55555555_5755f5ff)
@@
 	(footprint "Capacitor_THT:C_Disc_D5.0mm_W2.5mm_P2.50mm"
 		(layer "F.Cu")
-		(at 109.22 143.51)
+		(at 111.145 118.745)
 		(descr "C, Disc series, Radial, pin pitch=2.50mm, diameter*width=5*2.5mm^2, Capacitor, http://cdn-reichelt.de/documents/datenblatt/B300/DS_KERKO_TC.pdf")
 		(tags "C Disc series Radial pin pitch 2.50mm diameter 5mm width 2.5mm Capacitor")
@@
 	)
 	(segment
-		(start 111.72 143.51)
-		(end 111.719999 132.120001)
+		(start 118.11 142.875)
+		(end 110.992767 142.875)
 		(width 0.5)
-		(layer "F.Cu")
+		(layer "B.Cu")
 		(net "+3V3")
 	)
 	(segment
-		(start 113.03 122.555)
-		(end 114.305 122.555)
+		(start 139.065 142.875)
+		(end 118.11 142.875)
 		(width 0.5)
-		(layer "F.Cu")
+		(layer "B.Cu")
 		(net "+3V3")
 	)
 	(segment
-		(start 146.05 135.89)
-		(end 139.065 142.875)
+		(start 110.992767 142.875)
+		(end 107.202767 139.085)
 		(width 0.5)
-		(layer "F.Cu")
+		(layer "B.Cu")
 		(net "+3V3")
 	)
 	(segment
-		(start 111.76 123.825)
-		(end 113.03 122.555)
+		(start 114.305 122.555)
+		(end 114.305 119.405)
 		(width 0.5)
-		(layer "F.Cu")
+		(layer "B.Cu")
 		(net "+3V3")
 	)
 	(segment
-		(start 139.065 142.875)
-		(end 118.11 142.875)
+		(start 112.395 117.495)
+		(end 109.648122 117.495)
 		(width 0.5)
-		(layer "F.Cu")
+		(layer "B.Cu")
 		(net "+3V3")
 	)
-	(via
-		(at 111.76 123.825)
-		(size 0.6)
-		(drill 0.3)
-		(layers "F.Cu" "B.Cu")
+	(segment
+		(start 105.435 138.312767)
+		(end 105.435 121.708122)
+		(width 0.5)
+		(layer "B.Cu")
 		(net "+3V3")
 	)
-	(via
-		(at 111.719999 132.120001)
-		(size 0.6)
-		(drill 0.3)
-		(layers "F.Cu" "B.Cu")
+	(segment
+		(start 107.202767 139.085)
+		(end 106.207233 139.085)
+		(width 0.5)
+		(layer "B.Cu")
+		(net "+3V3")
+	)
+	(segment
+		(start 146.05 135.89)
+		(end 139.065 142.875)
+		(width 0.5)
+		(layer "B.Cu")
 		(net "+3V3")
 	)
 	(segment
-		(start 117.475 143.51)
-		(end 111.72 143.51)
+		(start 109.648122 117.495)
+		(end 105.435 121.708122)
 		(width 0.5)
 		(layer "B.Cu")
@@
 	)
 	(segment
-		(start 111.76 123.825)
-		(end 111.76 132.08)
+		(start 106.207233 139.085)
+		(end 105.435 138.312767)
 		(width 0.5)
 		(layer "B.Cu")
@@
 	)
 	(segment
-		(start 118.11 142.875)
-		(end 117.475 143.51)
+		(start 114.305 119.405)
+		(end 113.645 118.745)
 		(width 0.5)
 		(layer "B.Cu")
@@
 	)
 	(segment
-		(start 111.76 132.08)
-		(end 111.719999 132.120001)
+		(start 113.645 118.745)
+		(end 112.395 117.495)
 		(width 0.5)
 		(layer "B.Cu")
@@
 	)
 	(segment
-		(start 109.22 143.51)
-		(end 110.47 144.76)
-		(width 0.5)
-		(layer "F.Cu")
-		(net "GND")
-	)
-	(segment
-		(start 110.49 125.095)
-		(end 114.305 125.095)
-		(width 0.5)
-		(layer "F.Cu")
-		(net "GND")
-	)
-	(segment
-		(start 146.05 138.43)
-		(end 140.335 144.145)
-		(width 0.5)
-		(layer "F.Cu")
-		(net "GND")
-	)
-	(segment
-		(start 112.852766 144.145)
-		(end 112.306383 144.691383)
-		(width 0.5)
-		(layer "F.Cu")
-		(net "GND")
-	)
-	(segment
-		(start 113.665 144.145)
-		(end 113.257233 144.145)
-		(width 0.5)
-		(layer "F.Cu")
-		(net "GND")
-	)
-	(segment
 		(start 146.05 138.43)
 		(end 148.59 138.43)
@@
 	)
 	(segment
-		(start 140.335 144.145)
-		(end 113.665 144.145)
-		(width 0.5)
-		(layer "F.Cu")
-		(net "GND")
-	)
-	(segment
 		(start 106.685 140.335)
 		(end 109.22 137.8)
@@
 	)
 	(segment
-		(start 113.665 144.145)
-		(end 112.852766 144.145)
-		(width 0.5)
-		(layer "F.Cu")
-		(net "GND")
-	)
-	(segment
-		(start 112.237767 144.76)
-		(end 112.306383 144.691383)
-		(width 0.5)
-		(layer "F.Cu")
-		(net "GND")
-	)
-	(segment
 		(start 109.22 137.8)
 		(end 109.22 128.905)
@@
 	)
 	(segment
-		(start 113.055 139.045)
-		(end 114.305 137.795)
-		(width 0.5)
-		(layer "F.Cu")
-		(net "GND")
-	)
-	(segment
-		(start 113.055 143.942767)
-		(end 113.055 139.045)
-		(width 0.5)
-		(layer "F.Cu")
-		(net "GND")
-	)
-	(segment
 		(start 156.21 138.43)
 		(end 158.75 138.43)
@@
 	)
 	(segment
-		(start 113.257233 144.145)
-		(end 113.055 143.942767)
-		(width 0.5)
-		(layer "F.Cu")
-		(net "GND")
-	)
-	(segment
-		(start 110.47 144.76)
-		(end 112.237767 144.76)
-		(width 0.5)
-		(layer "F.Cu")
-		(net "GND")
-	)
-	(segment
 		(start 151.13 138.43)
 		(end 153.67 138.43)
@@
 	)
 	(segment
-		(start 112.306383 144.691383)
-		(end 113.055 143.942767)
-		(width 0.5)
-		(layer "F.Cu")
-		(net "GND")
-	)
-	(segment
 		(start 153.67 138.43)
 		(end 156.21 138.43)
@@
 		(net "GND")
 	)
-	(via
-		(at 110.49 125.095)
-		(size 0.6)
-		(drill 0.3)
-		(layers "F.Cu" "B.Cu")
+	(segment
+		(start 140.355 144.125)
+		(end 146.05 138.43)
+		(width 0.5)
+		(layer "B.Cu")
 		(net "GND")
 	)
@@
 	)
 	(segment
+		(start 111.145 121.935)
+		(end 111.145 118.745)
+		(width 0.5)
+		(layer "B.Cu")
+		(net "GND")
+	)
+	(segment
+		(start 110.49 125.095)
+		(end 114.305 125.095)
+		(width 0.5)
+		(layer "B.Cu")
+		(net "GND")
+	)
+	(segment
 		(start 109.22 126.365)
 		(end 110.49 125.095)
@@
 	)
 	(segment
-		(start 109.22 142.87)
-		(end 106.685 140.335)
+		(start 110.475 144.125)
+		(end 140.355 144.125)
+		(width 0.5)
+		(layer "B.Cu")
+		(net "GND")
+	)
+	(segment
+		(start 106.685 140.335)
+		(end 110.475 144.125)
 		(width 0.5)
 		(layer "B.Cu")
@@
 	)
 	(segment
-		(start 109.22 143.51)
-		(end 109.22 142.87)
+		(start 114.305 125.095)
+		(end 111.145 121.935)
 		(width 0.5)
 		(layer "B.Cu")

Commit message: Fixed issues identified by Claude - batch 3
Routing:
- net GND: track 89.4 -> 17.8 mm, vias 1 -> 0
- net Net-(J1-ROW_3): track 196.2 -> 197.4 mm, vias 0 -> 4
- net /COL6: track 134.2 -> 133.1 mm, vias 2 -> 4
- net /COL7: track 112.0 -> 112.7 mm, vias 0 -> 4
- net /COL8: track 126.2 -> 126.6 mm, vias 0 -> 4
- net /COL1: track 53.1 -> 53.3 mm, vias 0 -> 2
- net Net-(J1-IN_PL): vias 0 -> 2
- net Net-(U1-Q7): vias 0 -> 1
- net /COL3: vias 0 -> 2
- net Net-(J1-ROW_1): vias 1 -> 3
- net +3V3: vias 0 -> 1
- net /COL5: vias 0 -> 2
- net Net-(J1-IN_CP): vias 0 -> 2
- net Net-(J1-ROW_2): vias 1 -> 3
- net /COL4: vias 0 -> 2
- added copper zone on B.Cu, net GND
- added copper zone on F.Cu, net GND

Commit message: Fixed issues identified by Claude - batch 4
Parts:
- D1, D10, D11, D12, D13, D14, D15, D16, D17, D18, D19, D2, D20, D21, D22, D23, D24, D3, D4, D5, D6, D7, D8, D9: value D -> D_Schottky; footprint Diode_SMD:D_SOD-123 -> Diode_SMD:D_SOD-323_HandSoldering
Routing:
- net /COL2: track 76.6 -> 77.0 mm, vias 0 -> 2

Commit message: Fixed issues identified by Claude - batch 5 - done
Parts:
- D1, D10, D11, D12, D13, D14, D15, D16, D17, D18, D19, D2, D20, D21, D22, D23, D24, D3, D4, D5, D6, D7, D8, D9: value D_Schottky -> SD103AWS
Routing:
- net GND: vias 0 -> 28
