File: PCBs/Shared_Main/Input_Shift_Register.kicad_sch (KiCad schematic)
At the start: 4 parts, among them J4 Screw_Terminal_01x08, U3 74HC165

Commit message: Renamed Right_Main to Shared_Main. Removed Left and System
Parts:
- C4: renamed from C2; footprint (none) -> Capacitor_THT:C_Disc_D5.0mm_W2.5mm_P2.50mm
- J10: renamed from J4; footprint (none) -> TerminalBlock_Phoenix:TerminalBlock_Phoenix_MPT-0,5-8-2.54_1x08_P2.54mm_Horizontal
- U4: renamed from U3; footprint (none) -> Package_DIP:DIP-16_W7.62mm
- renumbered RN2 to RN1

Commit message: shared main wip
Parts:
- J10: value Screw_Terminal_01x08 -> Digital inputs
Changed lines of the file:
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@@
 			)
 		)
-		(property "Value" "Screw_Terminal_01x08"
+		(property "Value" "Digital inputs"
 			(at 100.33 91.4399 0)
 			(show_name no)

Commit message: stuff
Connections:
- net +5V renamed +3V3
Changed lines of the file:
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@@
-	)
-	(symbol
-		(lib_id "power:+5V")
-		(at 116.84 58.42 0)
-		(unit 1)
-		(body_style 1)
-		(exclude_from_sim no)
-		(in_bom yes)
-		(on_board yes)
-		(in_pos_files yes)
-		(dnp no)
-		(fields_autoplaced yes)
-		(property "Reference" "#PWR026"
-			(at 116.84 62.23 0)
-			(hide yes)
-			(show_name no)
-			(do_not_autoplace no)
-			(effects
-				(font
-					(size 1.27 1.27)
-				)
-			)
-		)
-		(property "Value" "+5V"
-			(at 116.84 53.34 0)
-			(show_name no)
-			(do_not_autoplace no)
-			(effects
-				(font
-					(size 1.27 1.27)
-				)
-			)
-		)
-		(property "Footprint" ""
-			(at 116.84 58.42 0)
-			(hide yes)
-			(show_name no)
-			(do_not_autoplace no)
-			(effects
-				(font
-					(size 1.27 1.27)
-				)
-			)
-		)
-		(property "Datasheet" ""
-			(at 116.84 58.42 0)
-			(hide yes)
-			(show_name no)
-			(do_not_autoplace no)
-			(effects
-				(font
-					(size 1.27 1.27)
-				)
-			)
-		)
-		(property "Description" "Power symbol creates a global label with name \"+5V\""
-			(at 116.84 58.42 0)
-			(hide yes)
-			(show_name no)
-			(do_not_autoplace no)
-			(effects
-				(font
-					(size 1.27 1.27)
-				)
-			)
-		)
-		(pin "1"
-		)
-		(instances
-			(project "Shared_Main"
-				(path "/70ceab5e-e31b-4508-a755-c321a835a8c9/06890bf6-dd23-4e88-9f1e-ae85625d1e22"
-					(reference "#PWR036")
-					(unit 1)
-				)
-				(path "/70ceab5e-e31b-4508-a755-c321a835a8c9/1118328f-a1b2-4dcf-b1c5-36c97ae5f908"
-					(reference "#PWR026")
-					(unit 1)
-				)
-				(path "/70ceab5e-e31b-4508-a755-c321a835a8c9/689e04ea-9ab8-44cb-ac25-fd1df69ea6ca"
-					(reference "#PWR046")
-					(unit 1)
-				)
-				(path "/70ceab5e-e31b-4508-a755-c321a835a8c9/69476812-841e-42e1-9ee1-30f93f6ede61"
-					(reference "#PWR031")
-					(unit 1)
-				)
-				(path "/70ceab5e-e31b-4508-a755-c321a835a8c9/b184a816-d02f-4ef9-897c-d31b5b062636"
-					(reference "#PWR041")
-					(unit 1)
-				)
-				(path "/70ceab5e-e31b-4508-a755-c321a835a8c9/ffdc2058-e5d3-4693-94cd-ce1a8b4b8c8e"
-					(reference "#PWR051")
-					(unit 1)
-				)
-			)
-		)
 	)
 	(symbol
@@
 	)
 	(symbol
-		(lib_id "power:+5V")
+		(lib_id "power:+3V3")
 		(at 158.75 69.85 90)
 		(unit 1)
@@
 		(dnp no)
 		(fields_autoplaced yes)
-		(property "Reference" "#PWR028"
+		(property "Reference" "#PWR020"
 			(at 162.56 69.85 0)
 			(hide yes)
@@
 			)
 		)
-		(property "Value" "+5V"
+		(property "Value" "+3V3"
 			(at 154.94 69.8499 90)
 			(show_name no)
@@
 			)
 		)
-		(property "Description" "Power symbol creates a global label with name \"+5V\""
+		(property "Description" "Power symbol creates a global label with name \"+3V3\""
 			(at 158.75 69.85 0)
 			(hide yes)
@@
 			(project "Shared_Main"
 				(path "/70ceab5e-e31b-4508-a755-c321a835a8c9/06890bf6-dd23-4e88-9f1e-ae85625d1e22"
-					(reference "#PWR038")
+					(reference "#PWR023")
 					(unit 1)
 				)
 				(path "/70ceab5e-e31b-4508-a755-c321a835a8c9/1118328f-a1b2-4dcf-b1c5-36c97ae5f908"
+					(reference "#PWR020")
+					(unit 1)
+				)
+				(path "/70ceab5e-e31b-4508-a755-c321a835a8c9/689e04ea-9ab8-44cb-ac25-fd1df69ea6ca"
+					(reference "#PWR025")
+					(unit 1)
+				)
+				(path "/70ceab5e-e31b-4508-a755-c321a835a8c9/69476812-841e-42e1-9ee1-30f93f6ede61"
+					(reference "#PWR022")
+					(unit 1)
+				)
+				(path "/70ceab5e-e31b-4508-a755-c321a835a8c9/b184a816-d02f-4ef9-897c-d31b5b062636"
+					(reference "#PWR024")
+					(unit 1)
+				)
+				(path "/70ceab5e-e31b-4508-a755-c321a835a8c9/ffdc2058-e5d3-4693-94cd-ce1a8b4b8c8e"
 					(reference "#PWR028")
-					(unit 1)
-				)
-				(path "/70ceab5e-e31b-4508-a755-c321a835a8c9/689e04ea-9ab8-44cb-ac25-fd1df69ea6ca"
-					(reference "#PWR048")
-					(unit 1)
-				)
-				(path "/70ceab5e-e31b-4508-a755-c321a835a8c9/69476812-841e-42e1-9ee1-30f93f6ede61"
-					(reference "#PWR033")
-					(unit 1)
-				)
-				(path "/70ceab5e-e31b-4508-a755-c321a835a8c9/b184a816-d02f-4ef9-897c-d31b5b062636"
-					(reference "#PWR043")
-					(unit 1)
-				)
-				(path "/70ceab5e-e31b-4508-a755-c321a835a8c9/ffdc2058-e5d3-4693-94cd-ce1a8b4b8c8e"
-					(reference "#PWR053")
 					(unit 1)
 				)
@@
 					(unit 1)
 				)
+			)
+		)
+	)
+	(symbol
+		(lib_id "power:+3V3")
+		(at 116.84 58.42 0)
+		(unit 1)
+		(body_style 1)
+		(exclude_from_sim no)
+		(in_bom yes)
+		(on_board yes)
+		(in_pos_files yes)
+		(dnp no)
+		(fields_autoplaced yes)
+		(property "Reference" "#PWR026"
+			(at 116.84 62.23 0)
+			(hide yes)
+			(show_name no)
+			(do_not_autoplace no)
+			(effects
+				(font
+					(size 1.27 1.27)
+				)
+			)
+		)
+		(property "Value" "+3V3"
+			(at 116.84 53.34 0)
+			(show_name no)
+			(do_not_autoplace no)
+			(effects
+				(font
+					(size 1.27 1.27)
+				)
+			)
+		)
+		(property "Footprint" ""
+			(at 116.84 58.42 0)
+			(hide yes)
+			(show_name no)
+			(do_not_autoplace no)
+			(effects
+				(font
+					(size 1.27 1.27)
+				)
+			)
+		)
+		(property "Datasheet" ""
+			(at 116.84 58.42 0)
+			(hide yes)
+			(show_name no)
+			(do_not_autoplace no)
+			(effects
+				(font
+					(size 1.27 1.27)
+				)
+			)
+		)
+		(property "Description" "Power symbol creates a global label with name \"+3V3\""
+			(at 116.84 58.42 0)
+			(hide yes)
+			(show_name no)
+			(do_not_autoplace no)
+			(effects
+				(font
+					(size 1.27 1.27)
+				)
+			)
+		)
+		(pin "1"
+		)
+		(instances
+			(project "Shared_Main"
+				(path "/70ceab5e-e31b-4508-a755-c321a835a8c9/06890bf6-dd23-4e88-9f1e-ae85625d1e22"
+					(reference "#PWR033")
+					(unit 1)
+				)
+				(path "/70ceab5e-e31b-4508-a755-c321a835a8c9/1118328f-a1b2-4dcf-b1c5-36c97ae5f908"
+					(reference "#PWR026")
+					(unit 1)
+				)
+				(path "/70ceab5e-e31b-4508-a755-c321a835a8c9/689e04ea-9ab8-44cb-ac25-fd1df69ea6ca"
+					(reference "#PWR038")
+					(unit 1)
+				)
+				(path "/70ceab5e-e31b-4508-a755-c321a835a8c9/69476812-841e-42e1-9ee1-30f93f6ede61"
+					(reference "#PWR031")
+					(unit 1)
+				)
+				(path "/70ceab5e-e31b-4508-a755-c321a835a8c9/b184a816-d02f-4ef9-897c-d31b5b062636"
+					(reference "#PWR036")
+					(unit 1)
+				)
+				(path "/70ceab5e-e31b-4508-a755-c321a835a8c9/ffdc2058-e5d3-4693-94cd-ce1a8b4b8c8e"
+					(reference "#PWR041")
+					(unit 1)
+				)
