File: PCBs/Shared_Main/Input_Shift_Register.kicad_sch (KiCad schematic)
At the start: 4 parts, among them J10 Digital inputs, U4 74HC165

Commit message: Fix 74HC4051 enable, set pull-up values, name keypad column nets
Shared_Main:
- U2 (74HC4051) pin 6 (~E) was tied to +3V3, permanently inhibiting all
  eight analog channels. Moved to GND. The pad had no tracks on it, so
  the board change is just which plane claims it (In2 +3V3 -> In1 GND);
  all zones refilled.
- RN1-RN6 pull-up arrays had no value assigned (still reading the
  R_Network08 symbol default). Set to 10k, matching RN8. Board footprint
  value fields synced to match.
- Also includes graphical tidy-up of junction/wire placement (no netlist
  change).

Right_Keypad:
- RN1 pull-up array set to 10k, board field synced.
- U1 was using a locally modified 74HC165 whose D0-D3 pins had been moved
  (via Swap Pins) so the column rails fan out to RN1 without crossing.
  That recorded the bit-order decision in pin geometry, where nothing
  diffs it and an "Update Symbols from Library" would silently remap four
  nets. Reverted U1 to the stock 74xx:74HC165 and expressed the same
  mapping as named nets COL1-COL8 instead:

      COL1 -> D3   COL5 -> D4
      COL2 -> D2   COL6 -> D5
      COL3 -> D1   COL7 -> D6
      COL4 -> D0   COL8 -> D7

  Connectivity is unchanged - verified by diffing before/after netlists
  with net names stripped and each net's pin set sorted. No copper moved
  (363 segments, 8 vias, 57 footprints before and after); only net names
  changed on the board.

Both projects: ERC 0, DRC 0, 0 unconnected, 0 schematic parity issues.

Co-Authored-By: Claude Opus 5 <noreply@anthropic.com>
Parts:
- RN1: value R_Network08 -> 10k
Changed lines of the file:
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@@
 			)
 		)
-		(property "Value" "R_Network08"
+		(property "Value" "10k"
 			(at 137.16 65.0239 0)
 			(show_name no)
