File: PCBs/Shared_Main/Input_Shift_Register.kicad_sch (KiCad schematic)
At the start: 4 parts, among them J10 Digital inputs, U4 74HC165

Commit message: change to vertical spring terminals
Parts:
- J10: footprint TerminalBlock_Phoenix:TerminalBlock_Phoenix_MPT-0,5-8-2.54_1x08_P2.54mm_Horizontal -> Custom_Footprints:SpringTerminal_1x08_P2.54mm_Vertical
Changed lines of the file:
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@@
 			)
 		)
-		(property "Footprint" "TerminalBlock_Phoenix:TerminalBlock_Phoenix_MPT-0,5-8-2.54_1x08_P2.54mm_Horizontal"
+		(property "Footprint" "Custom_Footprints:SpringTerminal_1x08_P2.54mm_Vertical"
 			(at 102.87 88.9 0)
 			(hide yes)

Commit message: revert to horizontal screw terminals to save cost
Parts:
- J10: footprint Custom_Footprints:SpringTerminal_1x08_P2.54mm_Vertical -> TerminalBlock_Phoenix:TerminalBlock_Phoenix_MPT-0,5-8-2.54_1x08_P2.54mm_Horizontal
Changed lines of the file:
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@@
 			)
 		)
-		(property "Footprint" "Custom_Footprints:SpringTerminal_1x08_P2.54mm_Vertical"
+		(property "Footprint" "TerminalBlock_Phoenix:TerminalBlock_Phoenix_MPT-0,5-8-2.54_1x08_P2.54mm_Horizontal"
 			(at 102.87 88.9 0)
 			(hide yes)
