File: PCBs/Shared_Main/Shared_Main.kicad_pcb (KiCad board)
At the start: 4 copper layers, 195.6 x 55.9 mm, 43 parts, among them J1 +5V and GND, J10 Screw_Terminal_01x08, J11 Screw_Terminal_01x08, J12 Screw_Terminal_01x08, J13 Screw_Terminal_01x08, J14 Screw_Terminal_01x08, J15 Screw_Terminal_01x08, J16 Conn_RJ45_Right_To_Left, J3 Encoder inputs B, J4 Encoder inputs A, J5 Analog inputs, J7 Conn_Right_Keypad, J8 Rotary switchs' pin 1, U1 MCP23017_SP, U10 MAX485E, U2 ULN2003A, U4 74HC165, U5 74HC165, U6 74HC165, U7 74HC165, U8 74HC165, U9 74HC165

Commit message: shared main wip
Parts:
- removed A1: Arduino_Micro_Socket, arduino-library:Arduino_Micro_Socket
- removed J3: Encoder inputs B, TerminalBlock_Phoenix:TerminalBlock_Phoenix_MPT-0,5-8-2.54_1x08_P2.54mm_Horizontal
- removed J8: Rotary switchs' pin 1, TerminalBlock_Phoenix:TerminalBlock_Phoenix_MPT-0,5-7-2.54_1x07_P2.54mm_Horizontal
- removed R2: 15k, Resistor_THT:R_Axial_DIN0207_L6.3mm_D2.5mm_P7.62mm_Horizontal
- removed R3: 4.7k, Resistor_THT:R_Axial_DIN0207_L6.3mm_D2.5mm_P7.62mm_Horizontal
- removed U10: MAX485E, Package_DIP:DIP-8_W7.62mm
- added J2: Rotary switches pin 1, TerminalBlock_Phoenix:TerminalBlock_Phoenix_MPT-0,5-8-2.54_1x08_P2.54mm_Horizontal, F.Cu at (200.0, 69.2)
- added Q1: BC547, Package_TO_SOT_THT:TO-92_Inline, F.Cu at (150.5, 80.0)
- added Q2: BC547, Package_TO_SOT_THT:TO-92_Inline, F.Cu at (144.1, 80.0)
- added Q3: BC547, Package_TO_SOT_THT:TO-92_Inline, F.Cu at (137.8, 80.0)
- added Q4: BC547, Package_TO_SOT_THT:TO-92_Inline, F.Cu at (131.4, 80.0)
- added Q5: BC547, Package_TO_SOT_THT:TO-92_Inline, F.Cu at (150.5, 73.0)
- added Q6: BC547, Package_TO_SOT_THT:TO-92_Inline, F.Cu at (144.1, 73.0)
- added Q7: BC547, Package_TO_SOT_THT:TO-92_Inline, F.Cu at (137.8, 73.0)
- added Q8: BC547, Package_TO_SOT_THT:TO-92_Inline, F.Cu at (131.4, 73.0)
- added RN8: 10k, Resistor_THT:R_Array_SIP9, F.Cu at (152.4, 66.7)
- J1: value +5V and GND -> Power; footprint TerminalBlock_Phoenix:TerminalBlock_Phoenix_MPT-0,5-8-2.54_1x08_P2.54mm_Horizontal -> TerminalBlock_Phoenix:TerminalBlock_Phoenix_PT-1,5-3-5.0-H_1x03_P5.00mm_Horizontal
- J10, J11, J12, J13, J14, J15: value Screw_Terminal_01x08 -> Digital inputs
- J16: value Conn_RJ45_Right_To_Left -> To other side
- J4: value Encoder inputs A -> Aux; footprint TerminalBlock_Phoenix:TerminalBlock_Phoenix_MPT-0,5-8-2.54_1x08_P2.54mm_Horizontal -> Connector_PinHeader_2.54mm:PinHeader_1x10_P2.54mm_Vertical
- J5: footprint TerminalBlock_Phoenix:TerminalBlock_Phoenix_MPT-0,5-6-2.54_1x06_P2.54mm_Horizontal -> TerminalBlock_Phoenix:TerminalBlock_Phoenix_MPT-0,5-8-2.54_1x08_P2.54mm_Horizontal
- J7: value Conn_Right_Keypad -> Keypad
- R1: value 15k -> 10k
- U1: value MCP23017_SP -> ESP32-S3-ZERO; footprint Package_DIP:DIP-28_W7.62mm -> ESP32-S3-ZERO:MODULE_ESP32-S3-ZERO
- U2: value ULN2003A -> 74HC4051
- moved U1 103.9 mm to (111.1, 75.6), turned to 0 degrees
- moved J1 99.0 mm to (87.1, 68.6)
- moved J4 90.9 mm to (123.2, 90.2), turned to -90 degrees
- moved C1 74.1 mm to (192.4, 40.0)
- moved J5 60.4 mm to (225.4, 69.2), turned to 180 degrees
- moved U2 33.7 mm to (226.1, 79.4)
- moved R4 33.0 mm to (78.7, 82.5), turned to 0 degrees
- moved R5 21.7 mm to (78.7, 86.4), turned to 0 degrees
- moved R1 14.1 mm to (126.4, 73.0), turned to -90 degrees
- moved R6 10.9 mm to (78.7, 90.2), turned to 0 degrees
- moved C6 2.54 mm to (177.2, 99.7)
- moved C7 2.54 mm to (151.8, 99.7)
- moved J13 2.54 mm to (131.4, 111.8)
- moved U4 2.54 mm to (224.8, 95.2)
- moved U5 2.54 mm to (199.4, 95.2)
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Connections:
- net /Input register 6/DS renamed /SR_Q7_KP
- C1 pad 1: +5V -> GND
- C1 pad 2: GND -> +5V
- J1 pad 1: +5V -> +3V3
- J1 pad 2: +5V -> GND
- J16 pad 1: Net-(J16-485_A) -> /FROM_A
- J16 pad 2: Net-(J16-485_B) -> GND
- J16 pad 3: +5V -> /FROM_B
- J4 pad 1: Net-(J4-Pin_1) -> /SR_CP
- J4 pad 2: Net-(J4-Pin_2) -> /SR_PL
- J4 pad 3: Net-(J4-Pin_3) -> /AUX0
- J4 pad 4: Net-(J4-Pin_4) -> /AUX1
- J4 pad 5: Net-(J4-Pin_5) -> /AUX2
- J4 pad 6: Net-(J4-Pin_6) -> /AUX3
- J4 pad 7: Net-(J4-Pin_7) -> /AUX4
- J4 pad 8: Net-(J4-Pin_8) -> /ADDR2
- J7 pad 10: /Input register 1//PL -> /SR_PL
- J7 pad 12: Net-(J7-ROW_1) -> /ADDR0
- J7 pad 14: Net-(J7-ROW_2) -> /ADDR1
- J7 pad 16: Net-(J7-ROW_3) -> /ADDR2
- J7 pad 8: /Input register 1/CP -> /SR_CP
- R1 pad 1: Net-(A1-D3/SCL) -> Net-(Q1-B)
- R1 pad 2: +5V -> /ROT_PIN_1
- R4 pad 1: Net-(A1-PadD9) -> /ADDR0
- R4 pad 2: Net-(J7-ROW_1) -> Net-(U1-GP1)
- R5 pad 1: Net-(A1-PadD10) -> /ADDR1
- R5 pad 2: Net-(J7-ROW_2) -> Net-(U1-GP2)
- R6 pad 1: Net-(A1-PadD11) -> /ADDR2
- R6 pad 2: Net-(J7-ROW_3) -> Net-(U1-GP3)
- U1 pad 1: Net-(J3-Pin_1) -> Net-(U1-GP1)
- U1 pad 10: GND -> /AUX1
- U1 pad 11: unconnected-(U1-NC-Pad11) -> /AUX2
- U1 pad 12: Net-(A1-D3/SCL) -> /AUX3
- U1 pad 13: Net-(A1-D2/SDA) -> /AUX4
- U1 pad 2: Net-(J3-Pin_2) -> Net-(U1-GP2)
- U1 pad 3: Net-(J3-Pin_3) -> Net-(U1-GP3)
- U1 pad 4: Net-(J3-Pin_4) -> /A
- U1 pad 5: Net-(J3-Pin_5) -> /ROT_PIN_1
- U1 pad 6: Net-(J3-Pin_6) -> /SR_Q7
- U1 pad 7: Net-(J3-Pin_7) -> /SR_CP
- U1 pad 8: Net-(J3-Pin_8) -> /SR_PL
- U1 pad 9: +5V -> /AUX0
- U2 pad 1: Net-(U2-I1) -> Net-(J5-Pin_4)
- U2 pad 10: Net-(J8-Pin_1) -> /ADDR1
- U2 pad 11: Net-(J8-Pin_2) -> /ADDR0
- U2 pad 12: Net-(J8-Pin_3) -> Net-(J5-Pin_5)
- U2 pad 13: Net-(J8-Pin_4) -> Net-(J5-Pin_8)
- U2 pad 14: Net-(J8-Pin_5) -> Net-(J5-Pin_7)
- U2 pad 15: Net-(J8-Pin_6) -> Net-(J5-Pin_6)
- U2 pad 16: Net-(J8-Pin_7) -> +5V
- U2 pad 2: Net-(U2-I1) -> Net-(J5-Pin_2)
- U2 pad 3: Net-(U2-I1) -> /A
- U2 pad 4: Net-(U2-I1) -> Net-(J5-Pin_1)
- U2 pad 5: Net-(U2-I1) -> Net-(J5-Pin_3)
- U2 pad 6: Net-(U2-I1) -> +3V3
- U2 pad 7: Net-(U2-I1) -> GND
- U2 pad 9: unconnected-(U2-COM-Pad9) -> /ADDR2
- U4 pad 1: /Input register 1//PL -> /SR_PL
- U4 pad 2: /Input register 1/CP -> /SR_CP
- U4 pad 9: /Input register 1/Q7 -> /SR_Q7
- U5 pad 1: /Input register 1//PL -> /SR_PL
- U5 pad 2: /Input register 1/CP -> /SR_CP
- U6 pad 1: /Input register 1//PL -> /SR_PL
- U6 pad 2: /Input register 1/CP -> /SR_CP
- U7 pad 1: /Input register 1//PL -> /SR_PL
- U7 pad 2: /Input register 1/CP -> /SR_CP
- U8 pad 1: /Input register 1//PL -> /SR_PL
- U8 pad 2: /Input register 1/CP -> /SR_CP
- U9 pad 1: /Input register 1//PL -> /SR_PL
- U9 pad 2: /Input register 1/CP -> /SR_CP
Routing:
- net /Input register 1//PL: track 187.3 -> 0.00 mm, vias 2 -> 0
- net /Input register 1/CP: track 183.5 -> 0.00 mm, vias 1 -> 0
- net /SR_PL: track 0.00 -> 163.6 mm, vias 0 -> 1
- net /SR_CP: track 0.00 -> 159.9 mm, vias 0 -> 1
- net Net-(U2-I1): track 147.0 -> 0.00 mm, vias 2 -> 0
- net Net-(A1-D7_INT4): track 118.8 -> 0.00 mm, vias 3 -> 0
- net Net-(A1-D2/SDA): track 118.4 -> 0.00 mm, vias 1 -> 0
- net Net-(A1-D3/SCL): track 116.3 -> 0.00 mm, vias 1 -> 0
- net /Input register 1/Q7: track 89.7 -> 0.00 mm, vias 2 -> 0
- net Net-(A1-D1/TX): track 62.3 -> 0.00 mm
- net Net-(J3-Pin_8): track 61.0 -> 0.00 mm
- net Net-(J3-Pin_7): track 59.5 -> 0.00 mm
- net Net-(A1-D0/RX): track 59.3 -> 0.00 mm, vias 1 -> 0
- net Net-(J3-Pin_6): track 58.1 -> 0.00 mm
- net Net-(J3-Pin_5): track 56.6 -> 0.00 mm
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- added copper zone on In2.Cu, net +3V3
- removed copper zone on In2.Cu, net +5V
Other:
- board text removed: "+5"
- board text removed: "GND"

Commit message: stuff
Parts:
- added H1: M3, MountingHole:MountingHole_3.2mm_M3, F.Cu at (234.9, 67.9)
- added H2: M3, MountingHole:MountingHole_3.2mm_M3, F.Cu at (234.3, 114.3)
- added H3: M3, MountingHole:MountingHole_3.2mm_M3, F.Cu at (59.1, 114.3)
- added H4: M3, MountingHole:MountingHole_3.2mm_M3, F.Cu at (59.1, 68.6)
- added R2: 100, Resistor_THT:R_Axial_DIN0207_L6.3mm_D2.5mm_P7.62mm_Horizontal, F.Cu at (109.2, 76.8)
- added R3: 100, Resistor_THT:R_Axial_DIN0207_L6.3mm_D2.5mm_P7.62mm_Horizontal, F.Cu at (109.2, 73.0)
- J16: value To other side -> Other unit
- R4, R5, R6: value 470 -> 100
- moved C2 46.3 mm to (102.9, 72.4), turned to 90 degrees
- moved C1 42.2 mm to (201.3, 81.3), turned to 0 degrees
- moved Q8 40.5 mm to (171.4, 66.7), turned to -90 degrees
- moved Q7 33.7 mm to (171.4, 73.0), turned to -90 degrees
- moved Q4 32.9 mm to (162.6, 69.2), turned to 90 degrees
- moved R4 30.5 mm to (109.2, 80.6)
- moved R5 30.5 mm to (109.2, 84.5)
- moved R6 30.5 mm to (109.2, 88.3)
- moved Q6 28.0 mm to (171.4, 79.4), turned to -90 degrees
- moved R1 25.7 mm to (151.1, 80.0)
- moved Q3 25.2 mm to (162.6, 75.6), turned to 90 degrees
- moved Q5 24.5 mm to (171.4, 85.7), turned to -90 degrees
- moved RN8 21.1 mm to (154.9, 87.6), turned to 90 degrees
- moved U2 20.5 mm to (207.0, 87.0), turned to 90 degrees
- moved J4 19.7 mm to (142.9, 90.2), turned to 180 degrees
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Connections:
- C1 pad 2: +5V -> +3V3
- C4 pad 2: +5V -> +3V3
- C5 pad 2: +5V -> +3V3
- C6 pad 2: +5V -> +3V3
- C7 pad 2: +5V -> +3V3
- C8 pad 2: +5V -> +3V3
- C9 pad 2: +5V -> +3V3
- J16 pad 1: /FROM_A -> Net-(J16-FROM_A)
- J16 pad 3: /FROM_B -> Net-(J16-FROM_B)
- J7 pad 12: /ADDR0 -> /ADDR0_KP
- J7 pad 14: /ADDR1 -> /ADDR1_KP
- J7 pad 16: /ADDR2 -> /ADDR2_KP
- J7 pad 2: +5V -> +3V3
- R4 pad 1: /ADDR0 -> /ADDR0_KP
- R4 pad 2: Net-(U1-GP1) -> /ADDR0
- R5 pad 1: /ADDR1 -> /ADDR1_KP
- R5 pad 2: Net-(U1-GP2) -> /ADDR1
- R6 pad 1: /ADDR2 -> /ADDR2_KP
- R6 pad 2: Net-(U1-GP3) -> /ADDR2
- RN1 pad 1: +5V -> +3V3
- RN2 pad 1: +5V -> +3V3
- RN3 pad 1: +5V -> +3V3
- RN4 pad 1: +5V -> +3V3
- RN5 pad 1: +5V -> +3V3
- RN6 pad 1: +5V -> +3V3
- U1 pad 1: Net-(U1-GP1) -> /ADDR0
- U1 pad 2: Net-(U1-GP2) -> /ADDR1
- U1 pad 3: Net-(U1-GP3) -> /ADDR2
- U2 pad 16: +5V -> +3V3
- U4 pad 16: +5V -> +3V3
- U5 pad 16: +5V -> +3V3
- U6 pad 16: +5V -> +3V3
- U7 pad 16: +5V -> +3V3
- U8 pad 16: +5V -> +3V3
- U9 pad 16: +5V -> +3V3
Routing:
- net /ADDR2: track 23.0 -> 138.2 mm
- net /ADDR1: track 24.2 -> 135.7 mm
- net /ADDR0: track 25.5 -> 133.1 mm
- net /A: track 0.00 -> 97.5 mm, vias 0 -> 1
- net /SR_Q7: track 11.1 -> 96.4 mm, vias 0 -> 1
- net +5V: track 0.00 -> 60.2 mm
- net /ADDR0_KP: track 0.00 -> 56.8 mm
- net /ADDR1_KP: track 0.00 -> 55.5 mm
- net Net-(Q1-B): track 0.00 -> 54.6 mm
- net /ADDR2_KP: track 0.00 -> 54.2 mm
- net Net-(J2-Pin_8): track 0.00 -> 46.1 mm
- net Net-(J2-Pin_7): track 0.00 -> 41.2 mm, vias 0 -> 1
- net Net-(J16-FROM_B): track 0.00 -> 36.7 mm
- net Net-(J2-Pin_6): track 0.00 -> 36.1 mm, vias 0 -> 1
- net Net-(J16-FROM_A): track 0.00 -> 35.0 mm
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Other:
- board size 195.6 x 55.9 mm -> 185.4 x 55.9 mm

Commit message: wip
Parts:
- Q1, Q2, Q3, Q4, Q5, Q6, Q7, Q8: footprint Package_TO_SOT_THT:TO-92_Inline -> Package_TO_SOT_THT:TO-92_Inline_Wide
- moved C2 13.6 mm to (116.2, 69.8)
- moved R1 7.62 mm to (151.1, 87.6), turned to 90 degrees
- moved Q1 2.69 mm to (160.7, 86.4), turned to 0 degrees
- moved Q2 2.69 mm to (160.7, 80.0), turned to 0 degrees
- moved Q3 2.69 mm to (160.7, 73.7), turned to 0 degrees
- moved Q4 2.69 mm to (160.7, 67.3), turned to 0 degrees
- moved H1 0.90 mm to (234.3, 68.6)
- moved Q5 0.90 mm to (170.8, 86.4), turned to 0 degrees
- moved Q6 0.90 mm to (170.8, 80.0), turned to 0 degrees
- moved Q8 0.90 mm to (170.8, 67.3), turned to 0 degrees
- moved Q7 0.90 mm to (170.8, 73.7), turned to 0 degrees
Routing:
- net Net-(Q1-B): track 54.6 -> 72.2 mm, vias 0 -> 1
- net Net-(Q7-E): track 18.9 -> 25.4 mm, vias 0 -> 2
- net Net-(Q8-E): track 18.0 -> 23.1 mm, vias 0 -> 1
- net Net-(J2-Pin_4): track 25.3 -> 30.0 mm, vias 0 -> 2
- net +5V: track 60.2 -> 55.8 mm
- net Net-(Q6-E): track 20.5 -> 24.5 mm, vias 0 -> 2
- net Net-(Q5-E): track 22.8 -> 26.8 mm, vias 0 -> 2
- net Net-(Q3-E): track 10.5 -> 14.0 mm
- net Net-(Q1-E): track 7.88 -> 11.3 mm
- net Net-(Q2-E): track 8.94 -> 11.8 mm
- net Net-(J2-Pin_3): track 20.1 -> 22.6 mm, vias 0 -> 1
- net Net-(J2-Pin_5): track 31.4 -> 33.8 mm, vias 2 -> 0
- net Net-(J2-Pin_8): track 46.1 -> 48.0 mm, vias 0 -> 2
- net Net-(Q4-E): track 14.1 -> 15.8 mm
- net Net-(J2-Pin_6): track 36.1 -> 37.7 mm, vias 1 -> 2
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Other:
- board text added: "3V3 GND 5V"
