File: PCBs/Shared_Main/Shared_Main.kicad_pcb (KiCad board)
At the start: 4 copper layers, 185.4 x 55.9 mm, 53 parts, among them J1 Power, J10 Digital inputs, J11 Digital inputs, J12 Digital inputs, J13 Digital inputs, J14 Digital inputs, J15 Digital inputs, J16 Other unit, J2 Rotary switches pin 1, J4 Aux, J5 Analog inputs, J7 Keypad, Q1 BC547, Q2 BC547, Q3 BC547, Q4 BC547, Q5 BC547, Q6 BC547, Q7 BC547, Q8 BC547, U1 ESP32-S3-ZERO, U2 74HC4051, U4 74HC165, U5 74HC165, U6 74HC165, U7 74HC165, U8 74HC165, U9 74HC165

Commit message: Fix 74HC4051 enable, set pull-up values, name keypad column nets
Shared_Main:
- U2 (74HC4051) pin 6 (~E) was tied to +3V3, permanently inhibiting all
  eight analog channels. Moved to GND. The pad had no tracks on it, so
  the board change is just which plane claims it (In2 +3V3 -> In1 GND);
  all zones refilled.
- RN1-RN6 pull-up arrays had no value assigned (still reading the
  R_Network08 symbol default). Set to 10k, matching RN8. Board footprint
  value fields synced to match.
- Also includes graphical tidy-up of junction/wire placement (no netlist
  change).

Right_Keypad:
- RN1 pull-up array set to 10k, board field synced.
- U1 was using a locally modified 74HC165 whose D0-D3 pins had been moved
  (via Swap Pins) so the column rails fan out to RN1 without crossing.
  That recorded the bit-order decision in pin geometry, where nothing
  diffs it and an "Update Symbols from Library" would silently remap four
  nets. Reverted U1 to the stock 74xx:74HC165 and expressed the same
  mapping as named nets COL1-COL8 instead:

      COL1 -> D3   COL5 -> D4
      COL2 -> D2   COL6 -> D5
      COL3 -> D1   COL7 -> D6
      COL4 -> D0   COL8 -> D7

  Connectivity is unchanged - verified by diffing before/after netlists
  with net names stripped and each net's pin set sorted. No copper moved
  (363 segments, 8 vias, 57 footprints before and after); only net names
  changed on the board.

Both projects: ERC 0, DRC 0, 0 unconnected, 0 schematic parity issues.

Co-Authored-By: Claude Opus 5 <noreply@anthropic.com>
Parts:
- RN1, RN2, RN3, RN4, RN5, RN6: value R_Network08 -> 10k
Connections:
- U2 pad 6: +3V3 -> GND
Changed lines of the file:
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@@
 			)
 		)
-		(property "Value" "R_Network08"
+		(property "Value" "10k"
 			(at 11.43 2.31 0)
 			(layer "F.SilkS")
@@
 			)
 		)
-		(property "Value" "R_Network08"
+		(property "Value" "10k"
 			(at 11.43 2.31 0)
 			(layer "F.SilkS")
@@
 			)
 		)
-		(property "Value" "R_Network08"
+		(property "Value" "10k"
 			(at 11.43 2.31 0)
 			(layer "F.SilkS")
@@
 			)
 		)
-		(property "Value" "R_Network08"
+		(property "Value" "10k"
 			(at 11.43 2.31 0)
 			(layer "F.SilkS")
@@
 			)
 		)
-		(property "Value" "R_Network08"
+		(property "Value" "10k"
 			(at 11.43 2.31 0)
 			(layer "F.SilkS")
@@
 			)
 		)
-		(property "Value" "R_Network08"
+		(property "Value" "10k"
 			(at 11.43 2.31 0)
 			(layer "F.SilkS")
@@
 			(layers "*.Cu" "*.Mask")
 			(remove_unused_layers no)
-			(net "+3V3")
+			(net "GND")
 			(pinfunction "~{E}_6")
 			(pintype "input")
