File: PCBs/Shared_Main/Shared_Main.kicad_pcb (KiCad board)
At the start: 4 copper layers, 175.3 x 61 mm, 49 parts, among them J1 Power, J10 Digital inputs, J11 Digital inputs, J12 Digital inputs, J13 Digital inputs, J14 Digital inputs, J15 Digital inputs, J16 Other unit, J2 Screw_Terminal_01x04, J4 Aux, J5 Analog inputs, J7 Keypad, Q1 BC547, Q2 BC547, Q3 BC547, Q4 BC547, U1 ESP32-S3-ZERO, U2 74HC4051, U4 74HC165, U5 74HC165, U6 74HC165, U7 74HC165, U8 74HC165, U9 74HC165

Commit message: zone fixes etc
Parts:
- moved H3 2.62 mm to (68.6, 119.4)
- moved H2 2.62 mm to (233.7, 119.4)
- moved H4 0.64 mm to (68.6, 68.6)
- moved J16 0.64 mm to (102.2, 78.1)
- moved H1 0.63 mm to (233.7, 68.6)
Routing:
- net Net-(J2-Pin_4): track 9.04 -> 14.1 mm
- net Net-(J2-Pin_3): track 9.57 -> 14.7 mm
- net Net-(J2-Pin_2): track 11.7 -> 16.8 mm
- net Net-(J2-Pin_1): track 17.5 -> 22.6 mm
- net /SR_PL: track 187.3 -> 184.5 mm, vias 3 -> 2
- net +5V: track 54.6 -> 55.4 mm
Other:
- board text added: "0"
- board text added: "16"
- board text added: "24"
- board text added: "32"
- board text added: "40"
- board text added: "8"
Changed lines of the file:
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@@
 		(capping no)
 		(filling no)
-		(zone_defaults)
 		(pcbplotparams
 			(layerselection 0x00000000_00000000_55555555_5755f5ff)
@@
 			(unlocked yes)
 			(layer "F.SilkS")
+			(hide yes)
 			(effects
 				(font
@@
 	(footprint "MountingHole:MountingHole_3.2mm_M3"
 		(layer "F.Cu")
-		(at 69.215 116.84)
+		(at 68.58 119.38)
 		(descr "Mounting Hole 3.2mm, M3, no annular, generated by kicad-footprint-generator mountinghole.py")
 		(tags "mountinghole M3")
@@
 			(unlocked yes)
 			(layer "F.SilkS")
+			(hide yes)
 			(effects
 				(font
@@
 			(unlocked yes)
 			(layer "F.SilkS")
+			(hide yes)
 			(effects
 				(font
@@
 	(footprint "MountingHole:MountingHole_3.2mm_M3"
 		(layer "F.Cu")
-		(at 69.215 68.58)
+		(at 68.58 68.58)
 		(descr "Mounting Hole 3.2mm, M3, no annular, generated by kicad-footprint-generator mountinghole.py")
 		(tags "mountinghole M3")
@@
 	(footprint "MountingHole:MountingHole_3.2mm_M3"
 		(layer "F.Cu")
-		(at 234.315 68.58)
+		(at 233.68 68.58)
 		(descr "Mounting Hole 3.2mm, M3, no annular, generated by kicad-footprint-generator mountinghole.py")
 		(tags "mountinghole M3")
@@
 	(footprint "MountingHole:MountingHole_3.2mm_M3"
 		(layer "F.Cu")
-		(at 234.315 116.84)
+		(at 233.68 119.38)
 		(descr "Mounting Hole 3.2mm, M3, no annular, generated by kicad-footprint-generator mountinghole.py")
 		(tags "mountinghole M3")
@@
 			(unlocked yes)
 			(layer "F.SilkS")
+			(hide yes)
 			(effects
 				(font
@@
 			(unlocked yes)
 			(layer "F.SilkS")
+			(hide yes)
 			(effects
 				(font
@@
 			(unlocked yes)
 			(layer "F.SilkS")
+			(hide yes)
 			(effects
 				(font
@@
 	(footprint "Connector_RJ:RJ45_Amphenol_54602-x08_Horizontal"
 		(layer "F.Cu")
-		(at 102.235 77.47 180)
+		(at 102.235 78.105 180)
 		(descr "8 Pol Shallow Latch Connector, Modjack, RJ45 (https://cdn.amphenol-icc.com/media/wysiwyg/files/drawing/c-bmj-0102.pdf)")
 		(tags "RJ45")
@@
 	)
 	(gr_rect
-		(start 64.135 63.5)
-		(end 239.395 124.46)
+		(start 63.5 63.5)
+		(end 238.76 124.46)
 		(stroke
 			(width 0.05)
@@
 		(layer "Edge.Cuts")
 	)
+	(gr_text "0"
+		(at 78.74 123.19 0)
+		(layer "F.SilkS")
+		(effects
+			(font
+				(size 1 1)
+				(thickness 0.1)
+			)
+			(justify left bottom)
+		)
+	)
+	(gr_text "8"
+		(at 104.14 123.19 0)
+		(layer "F.SilkS")
+		(effects
+			(font
+				(size 1 1)
+				(thickness 0.1)
+			)
+			(justify left bottom)
+		)
+	)
 	(gr_text "3V3  GND  5V"
-		(at 107.315 65.405 0)
+		(at 108.585 81.28 0)
+		(layer "F.SilkS")
+		(effects
+			(font
+				(size 1 1)
+				(thickness 0.1)
+			)
+			(justify left bottom)
+		)
+	)
+	(gr_text "16"
+		(at 129.54 123.19 0)
+		(layer "F.SilkS")
+		(effects
+			(font
+				(size 1 1)
+				(thickness 0.1)
+			)
+			(justify left bottom)
+		)
+	)
+	(gr_text "24"
+		(at 154.94 123.19 0)
+		(layer "F.SilkS")
+		(effects
+			(font
+				(size 1 1)
+				(thickness 0.1)
+			)
+			(justify left bottom)
+		)
+	)
+	(gr_text "32"
+		(at 180.34 123.19 0)
+		(layer "F.SilkS")
+		(effects
+			(font
+				(size 1 1)
+				(thickness 0.1)
+			)
+			(justify left bottom)
+		)
+	)
+	(gr_text "40"
+		(at 205.74 123.19 0)
 		(layer "F.SilkS")
 		(effects
@@
 	)
 	(segment
+		(start 187.325 74.295)
+		(end 187.325 69.215)
+		(width 0.25)
+		(layer "B.Cu")
+		(net "Net-(J2-Pin_2)")
+	)
+	(segment
 		(start 171.45 85.09)
 		(end 166.37 80.01)
@@
 	)
 	(segment
+		(start 192.405 74.295)
+		(end 192.405 69.215)
+		(width 0.25)
+		(layer "B.Cu")
+		(net "Net-(J2-Pin_4)")
+	)
+	(segment
 		(start 183.955 83.625)
 		(end 177.8 77.47)
@@
 	)
 	(segment
-		(start 123.825 78.74)
+		(start 123.19 79.375)
 		(end 125.73 76.835)
 		(width 0.25)
@@
 	)
 	(segment
-		(start 100.965 78.74)
-		(end 123.825 78.74)
+		(start 99.695 78.105)
+		(end 100.965 79.375)
 		(width 0.25)
 		(layer "F.Cu")
@@
 	)
 	(segment
-		(start 99.695 77.47)
-		(end 100.965 78.74)
+		(start 100.965 79.375)
+		(end 123.19 79.375)
 		(width 0.25)
 		(layer "F.Cu")
@@
 	)
 	(segment
+		(start 184.785 74.295)
+		(end 184.785 69.215)
+		(width 0.25)
+		(layer "B.Cu")
+		(net "Net-(J2-Pin_1)")
+	)
+	(segment
 		(start 189.865 74.295)
 		(end 189.865 79.375)
@@
 	)
 	(segment
+		(start 189.865 74.295)
+		(end 189.865 69.215)
+		(width 0.25)
+		(layer "B.Cu")
+		(net "Net-(J2-Pin_3)")
+	)
+	(segment
 		(start 125.095 73.025)
 		(end 125.73 73.025)
@@
 	)
 	(segment
-		(start 102.235 77.47)
-		(end 121.285 77.47)
+		(start 102.235 78.105)
+		(end 120.65 78.105)
 		(width 0.25)
 		(layer "F.Cu")
@@
 	)
 	(segment
-		(start 121.285 77.47)
+		(start 120.65 78.105)
 		(end 125.73 73.025)
 		(width 0.25)
@@
 	)
 	(via
-		(at 125.73 94.75)
-		(size 0.7)
-		(drill 0.3)
-		(layers "F.Cu" "B.Cu")
-		(net "/SR_PL")
-	)
-	(via
 		(at 152.654 95.25)
 		(size 0.7)
@@
 	)
 	(segment
-		(start 123.19 95.25)
-		(end 125.23 95.25)
-		(width 0.25)
-		(layer "B.Cu")
-		(net "/SR_PL")
-	)
-	(segment
 		(start 99.06 96.52)
 		(end 121.92 96.52)
@@
 	)
 	(segment
-		(start 125.23 95.25)
-		(end 125.73 94.75)
-		(width 0.25)
-		(layer "B.Cu")
-		(net "/SR_PL")
-	)
-	(segment
 		(start 172.72 96.52)
 		(end 173.99 95.25)
@@
 	)
 	(segment
+		(start 108.585 75.565)
+		(end 113.665 75.565)
+		(width 0.8)
+		(layer "B.Cu")
+		(net "+5V")
+	)
+	(segment
 		(start 137.16 67.31)
 		(end 132.715 67.31)
@@
 	)
 	(segment
-		(start 98.425 80.01)
-		(end 97.794189 80.01)
+		(start 132.715 67.31)
+		(end 116.84 67.31)
 		(width 0.8)
 		(layer "B.Cu")
@@
 	)
 	(segment
-		(start 113.665 75.565)
-		(end 96.52 75.565)
+		(start 96.444189 79.295)
+		(end 95.805 79.295)
 		(width 0.8)
 		(layer "B.Cu")
@@
 	)
 	(segment
-		(start 95.805 78.66)
-		(end 94.615 77.47)
+		(start 94.615 78.105)
+		(end 97.79 74.93)
 		(width 0.8)
 		(layer "B.Cu")
@@
 	)
 	(segment
-		(start 132.715 67.31)
+		(start 115.57 68.58)
 		(end 116.84 67.31)
 		(width 0.8)
@@
 	)
 	(segment
-		(start 115.57 68.58)
-		(end 116.84 67.31)
+		(start 95.805 79.295)
+		(end 94.615 78.105)
 		(width 0.8)
 		(layer "B.Cu")
@@
 	)
 	(segment
-		(start 97.794189 80.01)
-		(end 96.444189 78.66)
+		(start 97.794189 80.645)
+		(end 96.444189 79.295)
 		(width 0.8)
 		(layer "B.Cu")
@@
 	)
 	(segment
-		(start 115.57 73.66)
-		(end 113.665 75.565)
+		(start 107.95 74.93)
+		(end 108.585 75.565)
 		(width 0.8)
 		(layer "B.Cu")
@@
 	)
 	(segment
-		(start 96.444189 78.66)
-		(end 95.805 78.66)
+		(start 97.79 74.93)
+		(end 107.95 74.93)
 		(width 0.8)
 		(layer "B.Cu")
@@
 	)
 	(segment
-		(start 96.52 75.565)
-		(end 94.615 77.47)
+		(start 98.425 80.645)
+		(end 97.794189 80.645)
+		(width 0.8)
+		(layer "B.Cu")
+		(net "+5V")
+	)
+	(segment
+		(start 113.665 75.565)
+		(end 115.57 73.66)
 		(width 0.8)
 		(layer "B.Cu")
@@
 		(polygon
 			(pts
-				(xy 64.77 64.77) (xy 64.77 112.395) (xy 73.66 112.395) (xy 73.66 120.142) (xy 230.505 120.142) (xy 230.505 64.77)
+				(xy 76.2 64.77) (xy 76.2 85.09) (xy 67.31 85.09) (xy 67.31 107.95) (xy 76.2 107.95) (xy 76.2 119.38)
+				(xy 231.14 119.38) (xy 231.14 64.77)
 			)
 		)
@@
 		(polygon
 			(pts
-				(xy 64.77 64.77) (xy 64.77 112.395) (xy 73.66 112.395) (xy 73.66 120.142) (xy 230.505 120.142) (xy 230.505 64.77)
+				(xy 76.2 64.77) (xy 76.2 85.09) (xy 67.31 85.09) (xy 67.31 107.95) (xy 76.2 107.95) (xy 76.2 119.38)
+				(xy 231.14 119.38) (xy 231.14 64.77)
 			)
 		)
@@
 		(polygon
 			(pts
-				(xy 64.77 120.142) (xy 230.505 120.142) (xy 230.505 64.77) (xy 64.77 64.77)
+				(xy 76.2 85.09) (xy 67.31 85.09) (xy 67.31 107.95) (xy 76.2 107.95) (xy 76.2 119.38) (xy 231.14 119.38)
+				(xy 231.14 64.77) (xy 76.2 64.77)
 			)
 		)
@@
 		(polygon
 			(pts
-				(xy 64.77 120.142) (xy 230.505 120.142) (xy 230.505 64.77) (xy 64.77 64.77)
+				(xy 76.2 85.09) (xy 67.31 85.094379) (xy 67.31 107.95) (xy 76.2 107.95) (xy 76.2 119.38) (xy 231.14 119.38)
+				(xy 231.14 64.77) (xy 76.2 64.77)
 			)
 		)
