File: PCBs/Shared_Main/Shared_Main.kicad_sch (KiCad schematic)
At the start: 18 parts, among them J1 Power, J16 Other unit, J4 Aux, J5 Analog inputs, J7 Keypad, U1 ESP32-S3-ZERO, U2 74HC4051

Commit message: change to vertical spring terminals
Parts:
- J1: footprint TerminalBlock_Phoenix:TerminalBlock_Phoenix_PT-1,5-3-5.0-H_1x03_P5.00mm_Horizontal -> Custom_Footprints:SpringTerminal_1x03_P2.54mm_Vertical
- J5: footprint TerminalBlock_Phoenix:TerminalBlock_Phoenix_MPT-0,5-8-2.54_1x08_P2.54mm_Horizontal -> Custom_Footprints:SpringTerminal_1x08_P2.54mm_Vertical
Changed lines of the file:
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@@
 			)
 		)
-		(property "Footprint" "TerminalBlock_Phoenix:TerminalBlock_Phoenix_MPT-0,5-8-2.54_1x08_P2.54mm_Horizontal"
+		(property "Footprint" "Custom_Footprints:SpringTerminal_1x08_P2.54mm_Vertical"
 			(at 66.04 111.76 0)
 			(hide yes)
@@
 			)
 		)
-		(property "Footprint" "TerminalBlock_Phoenix:TerminalBlock_Phoenix_PT-1,5-3-5.0-H_1x03_P5.00mm_Horizontal"
+		(property "Footprint" "Custom_Footprints:SpringTerminal_1x03_P2.54mm_Vertical"
 			(at 129.54 173.99 0)
 			(hide yes)

Commit message: revert to horizontal screw terminals to save cost
Parts:
- J1: footprint Custom_Footprints:SpringTerminal_1x03_P2.54mm_Vertical -> TerminalBlock_Phoenix:TerminalBlock_Phoenix_MKDS-1,5-3_1x03_P5.00mm_Horizontal
- J5: footprint Custom_Footprints:SpringTerminal_1x08_P2.54mm_Vertical -> TerminalBlock_Phoenix:TerminalBlock_Phoenix_MPT-0,5-8-2.54_1x08_P2.54mm_Horizontal
Changed lines of the file:
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@@
 			)
 		)
-		(property "Footprint" "Custom_Footprints:SpringTerminal_1x08_P2.54mm_Vertical"
+		(property "Footprint" "TerminalBlock_Phoenix:TerminalBlock_Phoenix_MPT-0,5-8-2.54_1x08_P2.54mm_Horizontal"
 			(at 66.04 111.76 0)
 			(hide yes)
@@
 			)
 		)
-		(property "Footprint" "Custom_Footprints:SpringTerminal_1x03_P2.54mm_Vertical"
+		(property "Footprint" "TerminalBlock_Phoenix:TerminalBlock_Phoenix_MKDS-1,5-3_1x03_P5.00mm_Horizontal"
 			(at 129.54 173.99 0)
 			(hide yes)
