File: PCBs/Shared_Main/Shared_Main.kicad_sch (KiCad schematic)
At the start: 18 parts, among them J1 Power, J16 Other unit, J4 Aux, J5 Analog inputs, J7 Keypad, U1 ESP32-S3-ZERO, U2 74HC4051

Commit message: stuff
Parts:
- C2: footprint Capacitor_THT:C_Disc_D5.0mm_W2.5mm_P2.50mm -> Capacitor_THT:C_Disc_D6.0mm_W4.4mm_P5.00mm
Changed lines of the file:
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@@
 			)
 		)
-		(property "Footprint" "Capacitor_THT:C_Disc_D5.0mm_W2.5mm_P2.50mm"
+		(property "Footprint" "Capacitor_THT:C_Disc_D6.0mm_W4.4mm_P5.00mm"
 			(at 187.96 88.9 0)
 			(hide yes)

Commit message: Fixed issues identified by Claude - batch 1
Parts:
- added C3: 100uF, Capacitor_THT:CP_Radial_D5.0mm_P2.00mm, symbol Device:C_Polarized_Small
- added F1: 0.5A, Fuse:Fuse_Bourns_MF-RHT050, symbol Device:Polyfuse_Small
- added R8: 10k, Resistor_THT:R_Axial_DIN0207_L6.3mm_D2.5mm_P7.62mm_Horizontal, symbol Device:R_Small
Connections:
- net +3V3: now also R8.2
- net +5V: now also C3.1, F1.2; no longer J16.4 (5V), J16.7 (5V)
- net GND: now also C3.2
- net SR_Q7_KP: now also R8.1
- new net +5V_RJ45: F1.1, J16.4 (5V), J16.7 (5V)

Commit message: Fixed issues identified by Claude - batch 2
Parts:
- added R10, R9: 47, Resistor_THT:R_Axial_DIN0207_L6.3mm_D2.5mm_P7.62mm_Horizontal, symbol Device:R_Small
Connections:
- net SR_CP: now also R10.2; no longer U1.7 (GP7)
- net SR_PL: now also R9.2; no longer U1.8 (GP8)
- new net: R9.1, U1.8 (GP8)
- new net: R10.1, U1.7 (GP7)
Changed lines of the file:
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@@
 	(wire
 		(pts
-			(xy 189.23 110.49) (xy 195.58 110.49)
-		)
-		(stroke
-			(width 0)
-			(type default)
-		)
-	)
-	(wire
-		(pts
 			(xy 81.28 93.98) (xy 81.28 96.52)
 		)
@@
 	(wire
 		(pts
-			(xy 189.23 113.03) (xy 195.58 113.03)
+			(xy 81.28 91.44) (xy 81.28 93.98)
 		)
 		(stroke
@@
 	(wire
 		(pts
-			(xy 81.28 91.44) (xy 81.28 93.98)
+			(xy 88.9 106.68) (xy 99.06 106.68)
 		)
 		(stroke
@@
 	(wire
 		(pts
-			(xy 88.9 106.68) (xy 99.06 106.68)
+			(xy 170.18 54.61) (xy 170.18 59.69)
 		)
 		(stroke
@@
 	(wire
 		(pts
-			(xy 170.18 54.61) (xy 170.18 59.69)
+			(xy 62.23 76.2) (xy 63.5 76.2)
 		)
 		(stroke
@@
 	(wire
 		(pts
-			(xy 62.23 76.2) (xy 63.5 76.2)
+			(xy 119.38 54.61) (xy 119.38 62.23)
 		)
 		(stroke
@@
 	(wire
 		(pts
-			(xy 119.38 54.61) (xy 119.38 62.23)
+			(xy 134.62 54.61) (xy 134.62 59.69)
 		)
 		(stroke
@@
 	(wire
 		(pts
-			(xy 134.62 54.61) (xy 134.62 59.69)
+			(xy 232.41 149.86) (xy 238.76 149.86)
 		)
 		(stroke
@@
 	(wire
 		(pts
-			(xy 232.41 149.86) (xy 238.76 149.86)
+			(xy 194.31 113.03) (xy 201.93 113.03)
 		)
 		(stroke
@@
 	(wire
 		(pts
+			(xy 194.31 110.49) (xy 201.93 110.49)
+		)
+		(stroke
+			(width 0)
+			(type default)
+		)
+	)
+	(wire
+		(pts
 			(xy 116.84 59.69) (xy 134.62 59.69)
 		)
@@
 	)
 	(label "SR_PL"
-		(at 195.58 113.03 180)
+		(at 201.93 113.03 180)
 		(effects
 			(font
@@
 	)
 	(label "SR_CP"
-		(at 195.58 110.49 180)
+		(at 201.93 110.49 180)
 		(effects
 			(font
@@
 	(symbol
 		(lib_id "Device:R_Small")
+		(at 191.77 113.03 90)
+		(unit 1)
+		(body_style 1)
+		(exclude_from_sim no)
+		(in_bom yes)
+		(on_board yes)
+		(in_pos_files yes)
+		(dnp no)
+		(property "Reference" "R9"
+			(at 191.77 107.95 90)
+			(hide yes)
+			(show_name no)
+			(do_not_autoplace no)
+			(effects
+				(font
+					(size 1.016 1.016)
+				)
+			)
+		)
+		(property "Value" "47"
+			(at 191.77 113.03 90)
+			(show_name no)
+			(do_not_autoplace no)
+			(effects
+				(font
+					(size 1.27 1.27)
+				)
+			)
+		)
+		(property "Footprint" "Resistor_THT:R_Axial_DIN0207_L6.3mm_D2.5mm_P7.62mm_Horizontal"
+			(at 191.77 113.03 0)
+			(hide yes)
+			(show_name no)
+			(do_not_autoplace no)
+			(effects
+				(font
+					(size 1.27 1.27)
+				)
+			)
+		)
+		(property "Datasheet" ""
+			(at 191.77 113.03 0)
+			(hide yes)
+			(show_name no)
+			(do_not_autoplace no)
+			(effects
+				(font
+					(size 1.27 1.27)
+				)
+			)
+		)
+		(property "Description" "Resistor, small symbol"
+			(at 191.77 113.03 0)
+			(hide yes)
+			(show_name no)
+			(do_not_autoplace no)
+			(effects
+				(font
+					(size 1.27 1.27)
+				)
+			)
+		)
+		(pin "2"
+		)
+		(pin "1"
+		)
+		(instances
+			(project "Shared_Main"
+				(path "/70ceab5e-e31b-4508-a755-c321a835a8c9"
+					(reference "R9")
+					(unit 1)
+				)
+			)
+		)
+	)
+	(symbol
+		(lib_id "Device:R_Small")
 		(at 220.98 49.53 180)
 		(unit 1)
@@
 					(unit 1)
 				)
+			)
+		)
+	)
+	(symbol
+		(lib_id "Device:R_Small")
+		(at 191.77 110.49 90)
+		(unit 1)
+		(body_style 1)
+		(exclude_from_sim no)
+		(in_bom yes)
+		(on_board yes)
+		(in_pos_files yes)
+		(dnp no)
+		(property "Reference" "R10"
+			(at 191.77 105.41 90)
+			(hide yes)
+			(show_name no)
+			(do_not_autoplace no)
+			(effects
+				(font
+					(size 1.016 1.016)
+				)
+			)
+		)
+		(property "Value" "47"
+			(at 191.77 110.49 90)
+			(show_name no)
+			(do_not_autoplace no)
+			(effects
+				(font
+					(size 1.27 1.27)
+				)
+			)
+		)
+		(property "Footprint" "Resistor_THT:R_Axial_DIN0207_L6.3mm_D2.5mm_P7.62mm_Horizontal"
+			(at 191.77 110.49 0)
+			(hide yes)
+			(show_name no)
+			(do_not_autoplace no)
+			(effects
+				(font
+					(size 1.27 1.27)
+				)
+			)
+		)
+		(property "Datasheet" ""
+			(at 191.77 110.49 0)
+			(hide yes)
+			(show_name no)
+			(do_not_autoplace no)
+			(effects
+				(font
+					(size 1.27 1.27)
+				)
+			)
+		)
+		(property "Description" "Resistor, small symbol"
+			(at 191.77 110.49 0)
+			(hide yes)
+			(show_name no)
+			(do_not_autoplace no)
+			(effects
+				(font
+					(size 1.27 1.27)
+				)
+			)
+		)
+		(pin "2"
+		)
+		(pin "1"
+		)
+		(instances
+			(project "Shared_Main"
+				(path "/70ceab5e-e31b-4508-a755-c321a835a8c9"
+					(reference "R10")
+					(unit 1)
+				)
